File: boards/can-ssr/hardware/can-ssr.kicad_pcb (KiCad board)
At the start: 2 copper layers, 100 x 100 mm, 127 parts, among them J1 CAN IN, J2 CAN OUT, J3 ICSP, J30 MEAN WELL, J4 UART, Q1 IPB110N20N3LF, Q2 IPB110N20N3LF, Q20 2N7002, Q21 2N7002, Q22 2N7002, Q23 2N7002, Q24 2N7002, Q3 IPB110N20N3LF, Q4 IPB110N20N3LF, Q5 MMBT2907A, SW1 ADDR, U1 R-78E5.0-1.0, U10 VOM1271T, U11 VOM1271T, U12 ACS770ECB-100U-PFF-T, U2 MCP2562FD-E/P, U20 LM393B, U3 PIC18F47Q84-I/PT, U30 UCC12050DVE, U31 ISO1640DWR, U32 MCP3426A0-E/SN, U33 MCP4725A0T-E/CH, U34 MCP4725A0T-E/CH, U35 TLP222A, U36 MCP3426A1-E/SN, U40 MAX7219CWG+, U41 CC56-12SRWA, Y1 16MHz

Commit message: Manual final placement
Parts:
- moved R3 2.00 mm to (186.0, 130.0)
- moved C34 0.54 mm to (157.0, 137.3)
Routing:
- net /CAN, power, MCU/ICSPDAT: track 117.6 -> 63.5 mm, vias 15 -> 2
- net MW_REMOTE: track 7.98 -> 51.5 mm, vias 3 -> 2
- net GND: track 63.2 -> 87.9 mm, vias 48 -> 53
- net +5V: track 330.0 -> 344.7 mm, vias 12 -> 14
- net /CAN, power, MCU/CAN_TX: track 53.0 -> 47.5 mm
- net GND_LOAD: track 25.6 -> 30.2 mm, vias 45 -> 24
- net TRIP_RST: track 58.9 -> 54.4 mm
- net ACS_ADC: track 57.2 -> 53.1 mm
- net ACS_OUT: track 54.1 -> 51.3 mm, vias 5 -> 3
- net /Overcurrent trip, gate drive/VTH: track 35.0 -> 32.4 mm
- net /CAN, power, MCU/CANL: track 71.1 -> 68.8 mm, vias 5 -> 3
- net /Load-side sense and supply control/RLY_A: track 9.68 -> 7.38 mm
- net /CAN, power, MCU/LED_STATUS: track 72.1 -> 74.4 mm
- net /CAN, power, MCU/V12_BUS: track 138.3 -> 136.5 mm
- net /Display/DIG1: track 50.1 -> 51.7 mm
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