File: boards/can-ssr/hardware/can-ssr.kicad_pcb (KiCad board)
At the start: 2 copper layers, 100 x 100 mm, 127 parts, among them J1 CAN IN, J2 CAN OUT, J3 ICSP, J30 MEAN WELL, J4 UART, Q1 IPB110N20N3LF, Q2 IPB110N20N3LF, Q20 2N7002, Q21 2N7002, Q22 2N7002, Q23 2N7002, Q24 2N7002, Q3 IPB110N20N3LF, Q4 IPB110N20N3LF, Q5 MMBT2907A, SW1 ADDR, U1 R-78E5.0-1.0, U10 VOM1271T, U11 VOM1271T, U12 ACS770ECB-100U-PFF-T, U2 MCP2562FD-E/P, U20 LM393B, U3 PIC18F47Q84-I/PT, U30 UCC12050DVE, U31 ISO1640DWR, U32 MCP3426A0-E/SN, U33 MCP4725A0T-E/CH, U34 MCP4725A0T-E/CH, U35 TLP222A, U36 MCP3426A1-E/SN, U40 MAX7219CWG+, U41 CC56-12SRWA, Y1 16MHz

Commit message: can-ssr: refs on silk, values on fab; return-bolt via rings; ref placement
- Footprint text back to the usual layout: Reference on silkscreen,
  Value on fab, on each part's own side (bottom parts had their text on
  the front layers, mirrored)
- Restored the 12-via rings around the S- and L- return bolts (H2/H4)
  removed by track/via cleanup
- Second stitching link for five bottom-plane islands that hung from a
  single via; removed a duplicate stacked GND_LOAD via at (144.3, 155.5)
- First-pass reference placement: 118 moved clear of pads and silk
  (some ICs' refs go inside the body outline); C21, C34, R23, MH2 left
  for manual placement
- DRC: no errors, no unconnected items

Co-Authored-By: Claude Opus 5.5 <noreply@anthropic.com>
Routing:
- net GND: track 87.9 -> 102.0 mm, vias 53 -> 57
- net GND_LOAD: track 30.2 -> 31.7 mm, vias 24 -> 48
