File: boards/can-ssr/hardware/can-ssr.kicad_pcb (KiCad board)
At the start: 2 copper layers, 100 x 100 mm, 201 parts, among them J1 CAN IN/OUT, J3 ICSP, J30 MEAN WELL, J4 UART, Q1 IPB110N20N3LF, Q2 IPB110N20N3LF, Q20 2N7002, Q21 2N7002, Q22 2N7002, Q23 2N7002, Q24 2N7002, Q3 IPB110N20N3LF, Q4 IPB110N20N3LF, Q5 MMBT2907A, SW1 ADDR, U1 R-78E5.0-1.0, U10 VOM1271T, U11 VOM1271T, U12 ACS770ECB-100U-PFF-T, U2 MCP2562FD-E/P, U20 LM393B, U3 PIC18F47Q84-I/PT, U30 UCC12050DVE, U31 ISO1640DWR, U32 MCP3426A0-E/SN, U33 MCP4725A0T-E/CH, U34 MCP4725A0T-E/CH, U35 TLP222A, U36 MCP3426A1-E/SN, U40 MAX7219CWG+, U41 CC56-12SRWA, Y1 16MHz

Commit message: can-ssr: STD MOSFET IPB110N20N3LF (discontinued) -> IPB107N20N3G
Infineon's listed successor, same D2PAK footprint, no layout change. It is a
standard OptiMOS 3 without the Linear FET's wide SOA, so STD is now
sequenced-only: firmware 0.3 refuses hot turn-on on STD as on HV. No other
200 V 3-pin D2PAK linear-mode FET fits (IXTA30N25L2 is 140 mOhm).

fab.py: MPN_FIXUPS maps schematic MPNs to orderable DigiKey part numbers
(SH-7010C -> SH-7010MC).

Co-Authored-By: Claude Opus 5.5 <noreply@anthropic.com>
Parts:
- Q1, Q2, Q3, Q4: value IPB110N20N3LF -> IPB107N20N3G
Changed lines of the file:
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@@
 			)
 		)
-		(property "Value" "IPB110N20N3LF"
+		(property "Value" "IPB107N20N3G"
 			(at 0 6.65 180)
 			(layer "F.Fab")
@@
 			)
 		)
-		(property "MPN" "IPB110N20N3LFATMA1"
+		(property "MPN" "IPB107N20N3GATMA1"
 			(at 0 0 180)
 			(layer "F.Fab")
@@
 			)
 		)
-		(property "Build" "HC: IPB021N10NM5LF2 / STD: IPB110N20N3LF / HV: IPB407N30N (all Infineon D2PAK)"
+		(property "Build" "HC: IPB021N10NM5LF2 / STD: IPB107N20N3G / HV: IPB407N30N (all Infineon D2PAK)"
 			(at 0 0 180)
 			(layer "F.Fab")
@@
 			)
 		)
-		(property "Value" "IPB110N20N3LF"
+		(property "Value" "IPB107N20N3G"
 			(at 0 6.65 0)
 			(layer "F.Fab")
@@
 			)
 		)
-		(property "MPN" "IPB110N20N3LFATMA1"
+		(property "MPN" "IPB107N20N3GATMA1"
 			(at 0 0 0)
 			(layer "F.Fab")
@@
 			)
 		)
-		(property "Build" "HC: IPB021N10NM5LF2 / STD: IPB110N20N3LF / HV: IPB407N30N (all Infineon D2PAK)"
+		(property "Build" "HC: IPB021N10NM5LF2 / STD: IPB107N20N3G / HV: IPB407N30N (all Infineon D2PAK)"
 			(at 0 0 0)
 			(layer "F.Fab")
@@
 			)
 		)
-		(property "Value" "IPB110N20N3LF"
+		(property "Value" "IPB107N20N3G"
 			(at 0 6.65 180)
 			(layer "F.Fab")
@@
 			)
 		)
-		(property "MPN" "IPB110N20N3LFATMA1"
+		(property "MPN" "IPB107N20N3GATMA1"
 			(at 0 0 180)
 			(layer "F.Fab")
@@
 			)
 		)
-		(property "Build" "HC: IPB021N10NM5LF2 / STD: IPB110N20N3LF / HV: IPB407N30N (all Infineon D2PAK)"
+		(property "Build" "HC: IPB021N10NM5LF2 / STD: IPB107N20N3G / HV: IPB407N30N (all Infineon D2PAK)"
 			(at 0 0 180)
 			(layer "F.Fab")
@@
 			)
 		)
-		(property "Value" "IPB110N20N3LF"
+		(property "Value" "IPB107N20N3G"
 			(at 0 6.65 0)
 			(layer "F.Fab")
@@
 			)
 		)
-		(property "MPN" "IPB110N20N3LFATMA1"
+		(property "MPN" "IPB107N20N3GATMA1"
 			(at 0 0 0)
 			(layer "F.Fab")
@@
 			)
 		)
-		(property "Build" "HC: IPB021N10NM5LF2 / STD: IPB110N20N3LF / HV: IPB407N30N (all Infineon D2PAK)"
+		(property "Build" "HC: IPB021N10NM5LF2 / STD: IPB107N20N3G / HV: IPB407N30N (all Infineon D2PAK)"
 			(at 0 0 0)
 			(layer "F.Fab")

Commit message: Move core, can-card, io-card, serial-card, can-ssr, probe-helper to rev B
Rev A went to PCBWay and is tagged revA. Rev B replaces parts the Mouser
BOM check flagged (obsolete, end of life, not recommended for new designs,
or not orderable) and swaps out-of-stock passives and diodes for in-stock
equivalents. Field-only changes, same footprints, no layout change; the
reference boards (can-controller, pic-module) get the same part numbers.
The rev A order lists (DigiKey, Mouser) carry the same substitutions; the
Mouser list leaves out the T821 box headers (bought from DigiKey).

docs/rev-b-changes.md lists every change and the rev B to-dos (MAX7219 is
obsolete and must be replaced). transfer/mouser-revA.xlsx (Mouser BOM
check) consumed.

Co-Authored-By: Claude Opus 5.5 <noreply@anthropic.com>
Parts:
- U12: value ACS770ECB-100U-PFF-T -> ACS770LCB-100U-PFF-T
- U35: value TLP222A -> TLP240A
- U41: value CC56-12SRWA -> CC56-12SURKWA

Commit message: Mouser cart: SQD50P04-09L P-FET, Diotec P6SMBJ15A TVS
Out of stock: Vishay SUD50P04-08-GE3 (core Q1) -> SQD50P04-09L_GE3 and
Littelfuse SMBJ15A (12 V input TVS) -> Diotec P6SMBJ15A, same footprints,
in core, can-ssr and the can-controller/pic-module references. Logged in
docs/rev-b-changes.md; order lists regenerated. The cart as ordered is
docs/orders/mouser-cart-2026-10-12.xls.

Co-Authored-By: Claude Opus 5.5 <noreply@anthropic.com>
Parts:
- D2: value SMBJ15A -> P6SMBJ15A
Changed lines of the file:
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@@
 			)
 		)
-		(property "Value" "SMBJ15A"
+		(property "Value" "P6SMBJ15A"
 			(at 0 3 90)
 			(layer "F.Fab")
@@
 			)
 		)
-		(property "Manufacturer" "Littelfuse"
+		(property "Manufacturer" "Diotec Semiconductor"
 			(at 0 0 90)
 			(layer "F.Fab")
@@
 			)
 		)
-		(property "MPN" "SMBJ15A"
+		(property "MPN" "P6SMBJ15A"
 			(at 0 0 90)
 			(layer "F.Fab")
