File: boards/can-ssr/hardware/power_path.kicad_sch (KiCad schematic)
At the start: 24 parts, among them Q1 IPB107N20N3G, Q2 IPB107N20N3G, Q3 IPB107N20N3G, Q4 IPB107N20N3G, Q5 MMBT2907A, U10 VOM1271T, U11 VOM1271T, U12 ACS770ECB-100U-PFF-T

Commit message: Move core, can-card, io-card, serial-card, can-ssr, probe-helper to rev B
Rev A went to PCBWay and is tagged revA. Rev B replaces parts the Mouser
BOM check flagged (obsolete, end of life, not recommended for new designs,
or not orderable) and swaps out-of-stock passives and diodes for in-stock
equivalents. Field-only changes, same footprints, no layout change; the
reference boards (can-controller, pic-module) get the same part numbers.
The rev A order lists (DigiKey, Mouser) carry the same substitutions; the
Mouser list leaves out the T821 box headers (bought from DigiKey).

docs/rev-b-changes.md lists every change and the rev B to-dos (MAX7219 is
obsolete and must be replaced). transfer/mouser-revA.xlsx (Mouser BOM
check) consumed.

Co-Authored-By: Claude Opus 5.5 <noreply@anthropic.com>
Parts:
- C10: MPN C3225X7R2J683K250AA -> C1210C683KBRACTU; Manufacturer TDK -> KEMET
- C11: MPN GRM21BR71H104KA01L -> C0805C104K5RACTU; Manufacturer Murata -> KEMET
- D10: MPN SMAZ15-E3/61 -> SMAZ15-13-F; Manufacturer Vishay -> Diodes Incorporated
- D12: MPN ES1J-E3/61T -> ES1J; Manufacturer Vishay -> onsemi
- D13: MPN ES3J-E3/57T -> ES3J; Manufacturer Vishay -> onsemi
- U12: value ACS770ECB-100U-PFF-T -> ACS770LCB-100U-PFF-T; MPN ACS770ECB-100U-PFF-T -> ACS770LCB-100U-PFF-T
Changed lines of the file:
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@@
 		(title "CAN SSR: power path")
 		(date "2026-10-04")
-		(rev "A")
+		(rev "B")
 	)
 	(text "LOAD SIDE (referenced to GND_LOAD = RET, the return bar = supply -V). Up to 200 V: keep 250 V working clearances;\nabout 6 mm creepage to anything on the CAN/logic side. Heavy nets (VIN, SRC, VOUT_SW, VOUT, RET)\nare busbar runs: mask-free top copper with a soldered copper bar."
@@
 			)
 		)
-		(property "Manufacturer" "Vishay"
+		(property "Manufacturer" "Diodes Incorporated"
 			(at 241.3 101.6 0)
 			(hide yes)
@@
 			)
 		)
-		(property "MPN" "SMAZ15-E3/61"
+		(property "MPN" "SMAZ15-13-F"
 			(at 241.3 101.6 0)
 			(hide yes)
@@
 			)
 		)
-		(property "Manufacturer" "TDK"
+		(property "Manufacturer" "KEMET"
 			(at 223.52 177.8 0)
 			(hide yes)
@@
 			)
 		)
-		(property "MPN" "C3225X7R2J683K250AA"
+		(property "MPN" "C1210C683KBRACTU"
 			(at 223.52 177.8 0)
 			(hide yes)
@@
 			)
 		)
-		(property "Manufacturer" "Vishay"
+		(property "Manufacturer" "onsemi"
 			(at 241.3 190.5 0)
 			(hide yes)
@@
 			)
 		)
-		(property "MPN" "ES1J-E3/61T"
+		(property "MPN" "ES1J"
 			(at 241.3 190.5 0)
 			(hide yes)
@@
 			)
 		)
-		(property "Value" "ACS770ECB-100U-PFF-T"
+		(property "Value" "ACS770LCB-100U-PFF-T"
 			(at 309.88 180.34 0)
 			(effects
@@
 			)
 		)
-		(property "MPN" "ACS770ECB-100U-PFF-T"
+		(property "MPN" "ACS770LCB-100U-PFF-T"
 			(at 304.8 167.64 0)
 			(hide yes)
@@
 			)
 		)
-		(property "Manufacturer" "Murata"
+		(property "Manufacturer" "KEMET"
 			(at 330.2 160.02 0)
 			(hide yes)
@@
 			)
 		)
-		(property "MPN" "GRM21BR71H104KA01L"
+		(property "MPN" "C0805C104K5RACTU"
 			(at 330.2 160.02 0)
 			(hide yes)
@@
 			)
 		)
-		(property "Manufacturer" "Vishay"
+		(property "Manufacturer" "onsemi"
 			(at 152.4 152.4 0)
 			(hide yes)
@@
 			)
 		)
-		(property "MPN" "ES3J-E3/57T"
+		(property "MPN" "ES3J"
 			(at 152.4 152.4 0)
 			(hide yes)
