File: boards/can-ssr/hardware/display.kicad_sch (KiCad schematic)
At the start: 7 parts, among them U40 MAX7219CWG+, U41 CC56-12SRWA

Commit message: can-ssr: PCB synced from schematic; return bar on the bottom side
- tools/sync_pcb.py: update a board's PCB from its schematic (adds and
  links footprints, updates fields and nets, never deletes)
- can-ssr: all 123 footprints added (parked off the outline), parity clean
- Fix duplicate R40 (display RSET is now R50)
- Requirements: return bar bolted on the bottom side, bolt order
  S+ S- L- L+, via ring at S-/L-, single-point GND_LOAD

Co-Authored-By: Claude Opus 5.5 <noreply@anthropic.com>
Parts:
- removed R40: 27k, Resistor_SMD:R_1206_3216Metric_Pad1.30x1.75mm_HandSolder, symbol Device:R
- added R50: 27k, Resistor_SMD:R_1206_3216Metric_Pad1.30x1.75mm_HandSolder, symbol Device:R
Connections:
- net +5V: now also R50.1
- net ISET: now also R50.2
Changed lines of the file:
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@@
 		(instances
 			(project "can-ssr"
-				(path "/09b96810-cbdb-496a-83a0-e49ecf8d36fe/a92fac97-2063-4024-9634-4bf07e75ccbf"
+				(path "/09b96810-cbdb-496a-83a0-e49ecf8d36fe/be7c3673-9f9d-47bb-b8df-14533f74d1fd"
 					(reference "U40")
 					(unit 1)
@@
 		(instances
 			(project "can-ssr"
-				(path "/09b96810-cbdb-496a-83a0-e49ecf8d36fe/a92fac97-2063-4024-9634-4bf07e75ccbf"
+				(path "/09b96810-cbdb-496a-83a0-e49ecf8d36fe/be7c3673-9f9d-47bb-b8df-14533f74d1fd"
 					(reference "#PWR01")
 					(unit 1)
@@
 		(instances
 			(project "can-ssr"
-				(path "/09b96810-cbdb-496a-83a0-e49ecf8d36fe/a92fac97-2063-4024-9634-4bf07e75ccbf"
+				(path "/09b96810-cbdb-496a-83a0-e49ecf8d36fe/be7c3673-9f9d-47bb-b8df-14533f74d1fd"
 					(reference "#PWR02")
 					(unit 1)
@@
 		(instances
 			(project "can-ssr"
-				(path "/09b96810-cbdb-496a-83a0-e49ecf8d36fe/a92fac97-2063-4024-9634-4bf07e75ccbf"
+				(path "/09b96810-cbdb-496a-83a0-e49ecf8d36fe/be7c3673-9f9d-47bb-b8df-14533f74d1fd"
 					(reference "#PWR03")
 					(unit 1)
@@
 		(on_board yes)
 		(dnp no)
-		(property "Reference" "R40"
+		(property "Reference" "R50"
 			(at 68.58 74.93 0)
 			(effects
@@
 		(instances
 			(project "can-ssr"
-				(path "/09b96810-cbdb-496a-83a0-e49ecf8d36fe/a92fac97-2063-4024-9634-4bf07e75ccbf"
-					(reference "R40")
+				(path "/09b96810-cbdb-496a-83a0-e49ecf8d36fe/be7c3673-9f9d-47bb-b8df-14533f74d1fd"
+					(reference "R50")
 					(unit 1)
 				)
@@
 		(instances
 			(project "can-ssr"
-				(path "/09b96810-cbdb-496a-83a0-e49ecf8d36fe/a92fac97-2063-4024-9634-4bf07e75ccbf"
+				(path "/09b96810-cbdb-496a-83a0-e49ecf8d36fe/be7c3673-9f9d-47bb-b8df-14533f74d1fd"
 					(reference "#PWR04")
 					(unit 1)
@@
 		(instances
 			(project "can-ssr"
-				(path "/09b96810-cbdb-496a-83a0-e49ecf8d36fe/a92fac97-2063-4024-9634-4bf07e75ccbf"
+				(path "/09b96810-cbdb-496a-83a0-e49ecf8d36fe/be7c3673-9f9d-47bb-b8df-14533f74d1fd"
 					(reference "C43")
 					(unit 1)
@@
 		(instances
 			(project "can-ssr"
-				(path "/09b96810-cbdb-496a-83a0-e49ecf8d36fe/a92fac97-2063-4024-9634-4bf07e75ccbf"
+				(path "/09b96810-cbdb-496a-83a0-e49ecf8d36fe/be7c3673-9f9d-47bb-b8df-14533f74d1fd"
 					(reference "#PWR05")
 					(unit 1)
@@
 		(instances
 			(project "can-ssr"
-				(path "/09b96810-cbdb-496a-83a0-e49ecf8d36fe/a92fac97-2063-4024-9634-4bf07e75ccbf"
+				(path "/09b96810-cbdb-496a-83a0-e49ecf8d36fe/be7c3673-9f9d-47bb-b8df-14533f74d1fd"
 					(reference "#PWR06")
 					(unit 1)
@@
 		(instances
 			(project "can-ssr"
-				(path "/09b96810-cbdb-496a-83a0-e49ecf8d36fe/a92fac97-2063-4024-9634-4bf07e75ccbf"
+				(path "/09b96810-cbdb-496a-83a0-e49ecf8d36fe/be7c3673-9f9d-47bb-b8df-14533f74d1fd"
 					(reference "C44")
 					(unit 1)
@@
 		(instances
 			(project "can-ssr"
-				(path "/09b96810-cbdb-496a-83a0-e49ecf8d36fe/a92fac97-2063-4024-9634-4bf07e75ccbf"
+				(path "/09b96810-cbdb-496a-83a0-e49ecf8d36fe/be7c3673-9f9d-47bb-b8df-14533f74d1fd"
 					(reference "#PWR07")
 					(unit 1)
@@
 		(instances
 			(project "can-ssr"
-				(path "/09b96810-cbdb-496a-83a0-e49ecf8d36fe/a92fac97-2063-4024-9634-4bf07e75ccbf"
+				(path "/09b96810-cbdb-496a-83a0-e49ecf8d36fe/be7c3673-9f9d-47bb-b8df-14533f74d1fd"
 					(reference "#PWR08")
 					(unit 1)
@@
 		(instances
 			(project "can-ssr"
-				(path "/09b96810-cbdb-496a-83a0-e49ecf8d36fe/a92fac97-2063-4024-9634-4bf07e75ccbf"
+				(path "/09b96810-cbdb-496a-83a0-e49ecf8d36fe/be7c3673-9f9d-47bb-b8df-14533f74d1fd"
 					(reference "U41")
 					(unit 1)
@@
 		(instances
 			(project "can-ssr"
-				(path "/09b96810-cbdb-496a-83a0-e49ecf8d36fe/a92fac97-2063-4024-9634-4bf07e75ccbf"
+				(path "/09b96810-cbdb-496a-83a0-e49ecf8d36fe/be7c3673-9f9d-47bb-b8df-14533f74d1fd"
 					(reference "D40")
 					(unit 1)
@@
 		(instances
 			(project "can-ssr"
-				(path "/09b96810-cbdb-496a-83a0-e49ecf8d36fe/a92fac97-2063-4024-9634-4bf07e75ccbf"
+				(path "/09b96810-cbdb-496a-83a0-e49ecf8d36fe/be7c3673-9f9d-47bb-b8df-14533f74d1fd"
 					(reference "D41")
 					(unit 1)

Commit message: Move core, can-card, io-card, serial-card, can-ssr, probe-helper to rev B
Rev A went to PCBWay and is tagged revA. Rev B replaces parts the Mouser
BOM check flagged (obsolete, end of life, not recommended for new designs,
or not orderable) and swaps out-of-stock passives and diodes for in-stock
equivalents. Field-only changes, same footprints, no layout change; the
reference boards (can-controller, pic-module) get the same part numbers.
The rev A order lists (DigiKey, Mouser) carry the same substitutions; the
Mouser list leaves out the T821 box headers (bought from DigiKey).

docs/rev-b-changes.md lists every change and the rev B to-dos (MAX7219 is
obsolete and must be replaced). transfer/mouser-revA.xlsx (Mouser BOM
check) consumed.

Co-Authored-By: Claude Opus 5.5 <noreply@anthropic.com>
Parts:
- C43: MPN GRM21BR71H104KA01L -> C0805C104K5RACTU; Manufacturer Murata -> KEMET
- C44: MPN GRM31CR71E106KA12L -> CL31B106KAHNNNE; Manufacturer Murata -> Samsung Electro-Mechanics
- D40, D41: MPN LTST-C150GKT -> LTST-C150KGKT
- U41: value CC56-12SRWA -> CC56-12SURKWA; MPN CC56-12SRWA -> CC56-12SURKWA
Changed lines of the file:
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@@
 		(title "CAN SSR: display")
 		(date "2026-10-04")
-		(rev "A")
+		(rev "B")
 	)
 	(text "CAN/LOGIC SIDE. 4-digit 0.56 in red 7-segment readout, alternating V and A (V/A indicator LEDs);\nfault codes on a trip or build-resistor fault. MAX7219 multiplexes and current-limits, no segment resistors."
@@
 			)
 		)
-		(property "Manufacturer" "Murata"
+		(property "Manufacturer" "KEMET"
 			(at 63.5 139.7 0)
 			(hide yes)
@@
 			)
 		)
-		(property "MPN" "GRM21BR71H104KA01L"
+		(property "MPN" "C0805C104K5RACTU"
 			(at 63.5 139.7 0)
 			(hide yes)
@@
 			)
 		)
-		(property "Manufacturer" "Murata"
+		(property "Manufacturer" "Samsung Electro-Mechanics"
 			(at 83.82 139.7 0)
 			(hide yes)
@@
 			)
 		)
-		(property "MPN" "GRM31CR71E106KA12L"
+		(property "MPN" "CL31B106KAHNNNE"
 			(at 83.82 139.7 0)
 			(hide yes)
@@
 			)
 		)
-		(property "Value" "CC56-12SRWA"
+		(property "Value" "CC56-12SURKWA"
 			(at 190.5 115.57 0)
 			(effects
@@
 			)
 		)
-		(property "MPN" "CC56-12SRWA"
+		(property "MPN" "CC56-12SURKWA"
 			(at 190.5 96.52 0)
 			(hide yes)
@@
 			)
 		)
-		(property "MPN" "LTST-C150GKT"
+		(property "MPN" "LTST-C150KGKT"
 			(at 254 96.52 0)
 			(hide yes)
@@
 			)
 		)
-		(property "MPN" "LTST-C150GKT"
+		(property "MPN" "LTST-C150KGKT"
 			(at 271.78 96.52 0)
 			(hide yes)

Commit message: Rev B / rev A order: 10 uF CL31B106KAHZW6E, beads BLM31PG391SN1L
Both earlier substitutes (CL31B106KAHNNNE, BLM31KN102SH1L) are on
backorder at Mouser. CL31B106KAHZW6E has the same rating (1.4 mm tall).
The isolated-supply beads need no 1 kOhm: TI's reference uses 330 Ohm;
BLM31PG391SN1L is 390 Ohm @ 100 MHz, 2 A, 50 mOhm. Field-only changes;
order lists regenerated.

Co-Authored-By: Claude Opus 5.5 <noreply@anthropic.com>
Parts:
- C44: MPN CL31B106KAHNNNE -> CL31B106KAHZW6E
Changed lines of the file:
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@@
 			)
 		)
-		(property "MPN" "CL31B106KAHNNNE"
+		(property "MPN" "CL31B106KAHZW6E"
 			(at 83.82 139.7 0)
 			(hide yes)
