File: boards/can-ssr/hardware/load_side.kicad_sch (KiCad schematic)
At the start: 38 parts, among them J30 MEAN WELL, U30 UCC12050DVE, U31 ISO1640DWR, U32 MCP3428-E/SL, U33 MCP4725A0T-E/CH, U34 MCP4725A0T-E/CH, U35 TLP222A

Commit message: can-ssr: two MCP3426 and ~42 Hz filters for 100 Hz voltage sampling
Replace the shared MCP3428 with one MCP3426 per voltage (0x68 Vin + PV
readback, 0x69 Vout + PC readback), each converting continuously at
240 SPS, and lower the divider RC to ~42 Hz (470 nF). Reporting rate is
configurable, 10 Hz default, up to 100 Hz; requirements and READMEs
updated, fault capture noted as a planned firmware feature.

Co-Authored-By: Claude Opus 5.5 <noreply@anthropic.com>
Parts:
- removed U32: MCP3428-E/SL, Package_SO:SOIC-14_3.9x8.7mm_P1.27mm, symbol Analog_ADC:MCP3428x-xSL
- added C42: 100nF 50V X7R, Capacitor_SMD:C_0805_2012Metric_Pad1.18x1.45mm_HandSolder, symbol Device:C
- added U32: MCP3426A0-E/SN, Package_SO:SOIC-8_3.9x4.9mm_P1.27mm, symbol Analog_ADC:MCP3426Axx-xMS
- added U36: MCP3426A1-E/SN, Package_SO:SOIC-8_3.9x4.9mm_P1.27mm, symbol Analog_ADC:MCP3426Axx-xMS
- C37, C38: value 100nF 50V X7R -> 470nF 50V X7R; footprint Capacitor_SMD:C_0805_2012Metric_Pad1.18x1.45mm_HandSolder -> Capacitor_SMD:C_1206_3216Metric_Pad1.33x1.80mm_HandSolder; MPN GRM21BR71H104KA01L -> GRM31MR71H474KA01L
Connections:
- net GND_LOAD: now also C42.2, U32.2 (CH1-), U32.6 (V_{SS}), U32.8 (CH2-), U36.2 (CH1-), U36.6 (V_{SS}), U36.8 (CH2-)
- net PC_FB: now also U36.7 (CH2+)
- net PV_FB: now also U32.7 (CH2+)
- net SCL_ISO: now also U32.5 (SCL), U36.5 (SCL)
- net SDA_ISO: now also U32.4 (SDA), U36.4 (SDA)
- net V5_ISO: now also C42.1, U32.3 (V_{DD}), U36.3 (V_{DD})
- net VIN_DIV: now also U32.1 (CH1+)
- net VOUT_DIV: now also U36.1 (CH1+)
Other:
- note added: "Dividers: 3 x 332k (1206, 200 V each) over 8.06k = 1/124.6: 250 V -> 2.0 V full scale. 470 nF -> fc ~42 Hz anti-aliasing for 100 Hz reporting. MCP3426 input loading (~2 MOhm differential) is removed by calibration."
- note added: "I2C on the load side: MCP3426 0x68 / 0x69, MCP4725 0x60 (PV) / 0x61 (PC)."
- note added: "Two MCP3426 (2 ch, +/-2.048 V): U32 0x68 (A0 suffix) Vin + PV readback, U36 0x69 (A1) Vout + PC readback. Each converts its voltage continuously at 240 SPS (12 bit, ~0.125 V at 250 V FS): supports 100 Hz reporting; 10 Hz can average to finer resolution. Readbacks read occasionally."
- note removed: "Dividers: 3 x 332k (1206, 200 V each) over 8.06k = 1/124.6: 250 V -> 2.0 V full scale. 100 nF -> fc ~200 Hz anti-aliasing (sampled at 20 Hz, averaged). MCP3428 input loading (~2 MOhm differential) is removed by calibration."
- note removed: "I2C on the load side: MCP3428 0x68, MCP4725 0x60 (PV) and 0x61 (PC)."
- note removed: "MCP3428: 4 differential channels, +/-2.048 V, 16 bit at 15 SPS. CH1 Vin, CH2 Vout, CH3 PV readback, CH4 PC readback. Adr0/Adr1 low -> 0x68."

Commit message: Move core, can-card, io-card, serial-card, can-ssr, probe-helper to rev B
Rev A went to PCBWay and is tagged revA. Rev B replaces parts the Mouser
BOM check flagged (obsolete, end of life, not recommended for new designs,
or not orderable) and swaps out-of-stock passives and diodes for in-stock
equivalents. Field-only changes, same footprints, no layout change; the
reference boards (can-controller, pic-module) get the same part numbers.
The rev A order lists (DigiKey, Mouser) carry the same substitutions; the
Mouser list leaves out the T821 box headers (bought from DigiKey).

docs/rev-b-changes.md lists every change and the rev B to-dos (MAX7219 is
obsolete and must be replaced). transfer/mouser-revA.xlsx (Mouser BOM
check) consumed.

Co-Authored-By: Claude Opus 5.5 <noreply@anthropic.com>
Parts:
- C30, C32: MPN GRM31CR71E106KA12L -> CL31B106KAHNNNE; Manufacturer Murata -> Samsung Electro-Mechanics
- C31, C33, C34, C35, C36, C40, C41, C42: MPN GRM21BR71H104KA01L -> C0805C104K5RACTU; Manufacturer Murata -> KEMET
- C37, C38: MPN GRM31MR71H474KA01L -> C1206C474K5RACTU; Manufacturer Murata -> KEMET
- U35: value TLP222A -> TLP240A; MPN TLP222A(F) -> TLP240A(F)
Changed lines of the file:
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@@
 		(title "CAN SSR: load-side sense and Mean Well control")
 		(date "2026-10-04")
-		(rev "A")
+		(rev "B")
 	)
 	(text "Isolated load-side domain, referenced to GND_LOAD (return bar RET = supply -V). Powered and reached only\nthrough reinforced parts: U30 (UCC12050 DC/DC) and U31 (ISO1640 I2C). Keep ~6 mm creepage across them."
@@
 			)
 		)
-		(property "Manufacturer" "Murata"
+		(property "Manufacturer" "Samsung Electro-Mechanics"
 			(at 30.48 106.68 0)
 			(hide yes)
@@
 			)
 		)
-		(property "MPN" "GRM31CR71E106KA12L"
+		(property "MPN" "CL31B106KAHNNNE"
 			(at 30.48 106.68 0)
 			(hide yes)
@@
 			)
 		)
-		(property "Manufacturer" "Murata"
+		(property "Manufacturer" "KEMET"
 			(at 43.18 106.68 0)
 			(hide yes)
@@
 			)
 		)
-		(property "MPN" "GRM21BR71H104KA01L"
+		(property "MPN" "C0805C104K5RACTU"
 			(at 43.18 106.68 0)
 			(hide yes)
@@
 			)
 		)
-		(property "Manufacturer" "Murata"
+		(property "Manufacturer" "Samsung Electro-Mechanics"
 			(at 83.82 106.68 0)
 			(hide yes)
@@
 			)
 		)
-		(property "MPN" "GRM31CR71E106KA12L"
+		(property "MPN" "CL31B106KAHNNNE"
 			(at 83.82 106.68 0)
 			(hide yes)
@@
 			)
 		)
-		(property "Manufacturer" "Murata"
+		(property "Manufacturer" "KEMET"
 			(at 96.52 106.68 0)
 			(hide yes)
@@
 			)
 		)
-		(property "MPN" "GRM21BR71H104KA01L"
+		(property "MPN" "C0805C104K5RACTU"
 			(at 96.52 106.68 0)
 			(hide yes)
@@
 			)
 		)
-		(property "Manufacturer" "Murata"
+		(property "Manufacturer" "KEMET"
 			(at 30.48 190.5 0)
 			(hide yes)
@@
 			)
 		)
-		(property "MPN" "GRM21BR71H104KA01L"
+		(property "MPN" "C0805C104K5RACTU"
 			(at 30.48 190.5 0)
 			(hide yes)
@@
 			)
 		)
-		(property "Manufacturer" "Murata"
+		(property "Manufacturer" "KEMET"
 			(at 96.52 190.5 0)
 			(hide yes)
@@
 			)
 		)
-		(property "MPN" "GRM21BR71H104KA01L"
+		(property "MPN" "C0805C104K5RACTU"
 			(at 96.52 190.5 0)
 			(hide yes)
@@
 			)
 		)
-		(property "Manufacturer" "Murata"
+		(property "Manufacturer" "KEMET"
 			(at 205.74 48.26 0)
 			(hide yes)
@@
 			)
 		)
-		(property "MPN" "GRM21BR71H104KA01L"
+		(property "MPN" "C0805C104K5RACTU"
 			(at 205.74 48.26 0)
 			(hide yes)
@@
 			)
 		)
-		(property "Manufacturer" "Murata"
+		(property "Manufacturer" "KEMET"
 			(at 205.74 81.28 0)
 			(hide yes)
@@
 			)
 		)
-		(property "MPN" "GRM21BR71H104KA01L"
+		(property "MPN" "C0805C104K5RACTU"
 			(at 205.74 81.28 0)
 			(hide yes)
@@
 			)
 		)
-		(property "Manufacturer" "Murata"
+		(property "Manufacturer" "KEMET"
 			(at 205.74 139.7 0)
 			(hide yes)
@@
 			)
 		)
-		(property "MPN" "GRM31MR71H474KA01L"
+		(property "MPN" "C1206C474K5RACTU"
 			(at 205.74 139.7 0)
 			(hide yes)
@@
 			)
 		)
-		(property "Manufacturer" "Murata"
+		(property "Manufacturer" "KEMET"
 			(at 205.74 180.34 0)
 			(hide yes)
@@
 			)
 		)
-		(property "MPN" "GRM31MR71H474KA01L"
+		(property "MPN" "C1206C474K5RACTU"
 			(at 205.74 180.34 0)
 			(hide yes)
@@
 			)
 		)
-		(property "Manufacturer" "Murata"
+		(property "Manufacturer" "KEMET"
 			(at 254 48.26 0)
 			(hide yes)
@@
 			)
 		)
-		(property "MPN" "GRM21BR71H104KA01L"
+		(property "MPN" "C0805C104K5RACTU"
 			(at 254 48.26 0)
 			(hide yes)
@@
 			)
 		)
-		(property "Manufacturer" "Murata"
+		(property "Manufacturer" "KEMET"
 			(at 254 91.44 0)
 			(hide yes)
@@
 			)
 		)
-		(property "MPN" "GRM21BR71H104KA01L"
+		(property "MPN" "C0805C104K5RACTU"
 			(at 254 91.44 0)
 			(hide yes)
@@
 			)
 		)
-		(property "Value" "TLP222A"
+		(property "Value" "TLP240A"
 			(at 271.78 182.88 0)
 			(effects
@@
 			)
 		)
-		(property "MPN" "TLP222A(F)"
+		(property "MPN" "TLP240A(F)"
 			(at 271.78 175.26 0)
 			(hide yes)

Commit message: Rev B / rev A order: 10 uF CL31B106KAHZW6E, beads BLM31PG391SN1L
Both earlier substitutes (CL31B106KAHNNNE, BLM31KN102SH1L) are on
backorder at Mouser. CL31B106KAHZW6E has the same rating (1.4 mm tall).
The isolated-supply beads need no 1 kOhm: TI's reference uses 330 Ohm;
BLM31PG391SN1L is 390 Ohm @ 100 MHz, 2 A, 50 mOhm. Field-only changes;
order lists regenerated.

Co-Authored-By: Claude Opus 5.5 <noreply@anthropic.com>
Parts:
- C30, C32: MPN CL31B106KAHNNNE -> CL31B106KAHZW6E
Changed lines of the file:
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@@
 			)
 		)
-		(property "MPN" "CL31B106KAHNNNE"
+		(property "MPN" "CL31B106KAHZW6E"
 			(at 30.48 106.68 0)
 			(hide yes)
@@
 			)
 		)
-		(property "MPN" "CL31B106KAHNNNE"
+		(property "MPN" "CL31B106KAHZW6E"
 			(at 83.82 106.68 0)
 			(hide yes)
