File: boards/core/hardware/core.kicad_pcb (KiCad board)
At the start: 2 copper layers, 100 x 100 mm, 87 parts, among them J10 STACK BUS, J11 RACK 12V, J2 ICSP, J20 12V IN, J4 JD0-0004NL, J5 UART, Q1 SUD50P04-08, U1 PIC32MK1024MCM064-I/PT, U2 MCP1826S-3302E/DB, U20 TDN 5-2411WI, U3 W6100-L, Y1 12MHz, Y2 25MHz

Commit message: Core manual route
Routing:
- net /Ethernet/LNKn: track 0.00 -> 49.0 mm, vias 0 -> 2
- net SCL: track 34.7 -> 76.2 mm, vias 0 -> 2
- net /Ethernet/TXP: track 15.0 -> 38.9 mm, vias 0 -> 1
- net GND: track 346.7 -> 351.2 mm, vias 54 -> 55
- net RLY3: track 50.7 -> 48.0 mm
- net SDA: track 90.4 -> 92.7 mm
- net RLY1: track 98.1 -> 100.1 mm
- net DE1: track 92.4 -> 94.3 mm
- net RLY2: track 89.3 -> 91.2 mm
- net RLY4: track 91.3 -> 93.2 mm
- net /MCU/OSC2: track 11.8 -> 9.97 mm
- net U4RX: track 78.4 -> 80.2 mm
- net /Ethernet/XSCO: track 35.9 -> 34.2 mm
- net /Ethernet/RXP: track 41.8 -> 43.3 mm
- net /Ethernet/XSCI: track 21.4 -> 20.0 mm
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