File: boards/core/hardware/ethernet.kicad_sch (KiCad schematic)
At the start: 37 parts, among them J4 JD0-0004NL, U3 W6100-L, Y2 25MHz

Commit message: core: choose Y2/C29/C30/C31, start firmware (CAN card detect + 4 x CAN FD)
Parts: Y2 Abracon ABM3-25.000MHZ-D2Y-T (CL 18 pF) with 27 pF C0G load caps
(same as Y1), C29 Samsung CL31B335KAHVPNE 3.3 uF 25 V X7R. check_board clean.

Firmware (XC32 v5.00, PIC32MK-MC_DFP 1.13.270): 120 MHz via software clock
switch (errata DS80000898D 2.1.1), REFCLK4 40 MHz CAN clock, UART1 console,
W6100 reset/ID/PHY check, can-card detection from the ISOW1044 RXD idle
level, 4 x CAN FD (500k/2M default), loopback self-test.

Co-Authored-By: Claude Opus 5.5 <noreply@anthropic.com>
Parts:
- C29: MPN TBD (3.3 uF 25 V X7R 1206) -> CL31B335KAHVPNE; Manufacturer TBD -> Samsung Electro-Mechanics
- C30, C31: value 8pF 50V C0G -> 27pF 50V C0G; MPN TBD (8 pF 50 V C0G 0805, to suit the 25 MHz crystal) -> GRM2165C1H270JA01D; Manufacturer TBD -> Murata
- Y2: MPN TBD (25 MHz, 5032, CL 12 pF) -> ABM3-25.000MHZ-D2Y-T; Manufacturer TBD -> Abracon
Other:
- note added: "W6100 in SPI mode (MOD[3:0] = 0000) on SPI3. Support circuit per WIZnet W6100_Ref_Schematic_V110_use_mag: 2 x 49.9R + 0.1 uF per pair at the MDI pins, jack centre taps to 3V3A, beads 3V3D->3V3A and 1V2D->1V2A, RSET_BG 12k + 300R (12.3k 1 %), 25 MHz crystal (CL 18 pF) with 27 pF and 1M. The jack's magnetics isolate the host."
- note removed: "W6100 in SPI mode (MOD[3:0] = 0000) on SPI3. Support circuit per WIZnet W6100_Ref_Schematic_V110_use_mag: 2 x 49.9R + 0.1 uF per pair at the MDI pins, jack centre taps to 3V3A, beads 3V3D->3V3A and 1V2D->1V2A, RSET_BG 12k + 300R (12.3k 1 %), 25 MHz crystal with 8 pF and 1M. The jack's magnetics isolate the host."
Changed lines of the file:
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@@
 		(rev "A")
 	)
-	(text "W6100 in SPI mode (MOD[3:0] = 0000) on SPI3. Support circuit per WIZnet W6100_Ref_Schematic_V110_use_mag:\n2 x 49.9R + 0.1 uF per pair at the MDI pins, jack centre taps to 3V3A, beads 3V3D->3V3A and 1V2D->1V2A,\nRSET_BG 12k + 300R (12.3k 1 %), 25 MHz crystal with 8 pF and 1M. The jack's magnetics isolate the host."
+	(text "W6100 in SPI mode (MOD[3:0] = 0000) on SPI3. Support circuit per WIZnet W6100_Ref_Schematic_V110_use_mag:\n2 x 49.9R + 0.1 uF per pair at the MDI pins, jack centre taps to 3V3A, beads 3V3D->3V3A and 1V2D->1V2A,\nRSET_BG 12k + 300R (12.3k 1 %), 25 MHz crystal (CL 18 pF) with 27 pF and 1M. The jack's magnetics isolate the host."
 		(exclude_from_sim no)
 		(at 25.4 25.4 0)
@@
 			)
 		)
-		(property "Manufacturer" "TBD"
+		(property "Manufacturer" "Samsung Electro-Mechanics"
 			(at 241.3 55.88 0)
 			(hide yes)
@@
 			)
 		)
-		(property "MPN" "TBD (3.3 uF 25 V X7R 1206)"
+		(property "MPN" "CL31B335KAHVPNE"
 			(at 241.3 55.88 0)
 			(hide yes)
@@
 			)
 		)
-		(property "Manufacturer" "TBD"
+		(property "Manufacturer" "Abracon"
 			(at 254 190.5 0)
 			(hide yes)
@@
 			)
 		)
-		(property "MPN" "TBD (25 MHz, 5032, CL 12 pF)"
+		(property "MPN" "ABM3-25.000MHZ-D2Y-T"
 			(at 254 190.5 0)
 			(hide yes)
@@
 			)
 		)
-		(property "Value" "8pF 50V C0G"
+		(property "Value" "27pF 50V C0G"
 			(at 246.38 214.63 0)
 			(effects
@@
 			)
 		)
-		(property "Manufacturer" "TBD"
+		(property "Manufacturer" "Murata"
 			(at 243.84 213.36 0)
 			(hide yes)
@@
 			)
 		)
-		(property "MPN" "TBD (8 pF 50 V C0G 0805, to suit the 25 MHz crystal)"
+		(property "MPN" "GRM2165C1H270JA01D"
 			(at 243.84 213.36 0)
 			(hide yes)
@@
 			)
 		)
-		(property "Value" "8pF 50V C0G"
+		(property "Value" "27pF 50V C0G"
 			(at 266.7 214.63 0)
 			(effects
@@
 			)
 		)
-		(property "Manufacturer" "TBD"
+		(property "Manufacturer" "Murata"
 			(at 264.16 213.36 0)
 			(hide yes)
@@
 			)
 		)
-		(property "MPN" "TBD (8 pF 50 V C0G 0805, to suit the 25 MHz crystal)"
+		(property "MPN" "GRM2165C1H270JA01D"
 			(at 264.16 213.36 0)
 			(hide yes)

Commit message: Move core, can-card, io-card, serial-card, can-ssr, probe-helper to rev B
Rev A went to PCBWay and is tagged revA. Rev B replaces parts the Mouser
BOM check flagged (obsolete, end of life, not recommended for new designs,
or not orderable) and swaps out-of-stock passives and diodes for in-stock
equivalents. Field-only changes, same footprints, no layout change; the
reference boards (can-controller, pic-module) get the same part numbers.
The rev A order lists (DigiKey, Mouser) carry the same substitutions; the
Mouser list leaves out the T821 box headers (bought from DigiKey).

docs/rev-b-changes.md lists every change and the rev B to-dos (MAX7219 is
obsolete and must be replaced). transfer/mouser-revA.xlsx (Mouser BOM
check) consumed.

Co-Authored-By: Claude Opus 5.5 <noreply@anthropic.com>
Parts:
- C20, C21, C22, C23, C24, C25, C26, C27, C28, C32, C33, C34: MPN GRM21BR71H104KA01L -> C0805C104K5RACTU; Manufacturer Murata -> KEMET
- C30, C31: MPN GRM2165C1H270JA01D -> C0805C270J5GACTU; Manufacturer Murata -> KEMET
- C35: MPN GRM31MR71H105KA88L -> C1206C105K5RACTU; Manufacturer Murata -> KEMET
- R22, R23: MPN RC1206FR-07330RL -> RMCF1206FT330R; Manufacturer Yageo -> Stackpole
Changed lines of the file:
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@@
 		(title "Core: Ethernet (W6100)")
 		(date "2026-10-06")
-		(rev "A")
+		(rev "B")
 	)
 	(text "W6100 in SPI mode (MOD[3:0] = 0000) on SPI3. Support circuit per WIZnet W6100_Ref_Schematic_V110_use_mag:\n2 x 49.9R + 0.1 uF per pair at the MDI pins, jack centre taps to 3V3A, beads 3V3D->3V3A and 1V2D->1V2A,\nRSET_BG 12k + 300R (12.3k 1 %), 25 MHz crystal (CL 18 pF) with 27 pF and 1M. The jack's magnetics isolate the host."
@@
 			)
 		)
-		(property "Manufacturer" "Murata"
+		(property "Manufacturer" "KEMET"
 			(at 127 55.88 0)
 			(hide yes)
@@
 			)
 		)
-		(property "MPN" "GRM21BR71H104KA01L"
+		(property "MPN" "C0805C104K5RACTU"
 			(at 127 55.88 0)
 			(hide yes)
@@
 			)
 		)
-		(property "Manufacturer" "Murata"
+		(property "Manufacturer" "KEMET"
 			(at 139.7 55.88 0)
 			(hide yes)
@@
 			)
 		)
-		(property "MPN" "GRM21BR71H104KA01L"
+		(property "MPN" "C0805C104K5RACTU"
 			(at 139.7 55.88 0)
 			(hide yes)
@@
 			)
 		)
-		(property "Manufacturer" "Murata"
+		(property "Manufacturer" "KEMET"
 			(at 152.4 55.88 0)
 			(hide yes)
@@
 			)
 		)
-		(property "MPN" "GRM21BR71H104KA01L"
+		(property "MPN" "C0805C104K5RACTU"
 			(at 152.4 55.88 0)
 			(hide yes)
@@
 			)
 		)
-		(property "Manufacturer" "Murata"
+		(property "Manufacturer" "KEMET"
 			(at 165.1 55.88 0)
 			(hide yes)
@@
 			)
 		)
-		(property "MPN" "GRM21BR71H104KA01L"
+		(property "MPN" "C0805C104K5RACTU"
 			(at 165.1 55.88 0)
 			(hide yes)
@@
 			)
 		)
-		(property "Manufacturer" "Murata"
+		(property "Manufacturer" "KEMET"
 			(at 177.8 55.88 0)
 			(hide yes)
@@
 			)
 		)
-		(property "MPN" "GRM21BR71H104KA01L"
+		(property "MPN" "C0805C104K5RACTU"
 			(at 177.8 55.88 0)
 			(hide yes)
@@
 			)
 		)
-		(property "Manufacturer" "Murata"
+		(property "Manufacturer" "KEMET"
 			(at 190.5 55.88 0)
 			(hide yes)
@@
 			)
 		)
-		(property "MPN" "GRM21BR71H104KA01L"
+		(property "MPN" "C0805C104K5RACTU"
 			(at 190.5 55.88 0)
 			(hide yes)
@@
 			)
 		)
-		(property "Manufacturer" "Murata"
+		(property "Manufacturer" "KEMET"
 			(at 203.2 55.88 0)
 			(hide yes)
@@
 			)
 		)
-		(property "MPN" "GRM21BR71H104KA01L"
+		(property "MPN" "C0805C104K5RACTU"
 			(at 203.2 55.88 0)
 			(hide yes)
@@
 			)
 		)
-		(property "Manufacturer" "Murata"
+		(property "Manufacturer" "KEMET"
 			(at 215.9 55.88 0)
 			(hide yes)
@@
 			)
 		)
-		(property "MPN" "GRM21BR71H104KA01L"
+		(property "MPN" "C0805C104K5RACTU"
 			(at 215.9 55.88 0)
 			(hide yes)
@@
 			)
 		)
-		(property "Manufacturer" "Murata"
+		(property "Manufacturer" "KEMET"
 			(at 228.6 55.88 0)
 			(hide yes)
@@
 			)
 		)
-		(property "MPN" "GRM21BR71H104KA01L"
+		(property "MPN" "C0805C104K5RACTU"
 			(at 228.6 55.88 0)
 			(hide yes)
@@
 			)
 		)
-		(property "Manufacturer" "Murata"
+		(property "Manufacturer" "KEMET"
 			(at 243.84 213.36 0)
 			(hide yes)
@@
 			)
 		)
-		(property "MPN" "GRM2165C1H270JA01D"
+		(property "MPN" "C0805C270J5GACTU"
 			(at 243.84 213.36 0)
 			(hide yes)
@@
 			)
 		)
-		(property "Manufacturer" "Murata"
+		(property "Manufacturer" "KEMET"
 			(at 264.16 213.36 0)
 			(hide yes)
@@
 			)
 		)
-		(property "MPN" "GRM2165C1H270JA01D"
+		(property "MPN" "C0805C270J5GACTU"
 			(at 264.16 213.36 0)
 			(hide yes)
@@
 			)
 		)
-		(property "Manufacturer" "Murata"
+		(property "Manufacturer" "KEMET"
 			(at 294.64 129.54 0)
 			(hide yes)
@@
 			)
 		)
-		(property "MPN" "GRM21BR71H104KA01L"
+		(property "MPN" "C0805C104K5RACTU"
 			(at 294.64 129.54 0)
 			(hide yes)
@@
 			)
 		)
-		(property "Manufacturer" "Murata"
+		(property "Manufacturer" "KEMET"
 			(at 294.64 172.72 0)
 			(hide yes)
@@
 			)
 		)
-		(property "MPN" "GRM21BR71H104KA01L"
+		(property "MPN" "C0805C104K5RACTU"
 			(at 294.64 172.72 0)
 			(hide yes)
@@
 			)
 		)
-		(property "Manufacturer" "Murata"
+		(property "Manufacturer" "KEMET"
 			(at 330.2 228.6 0)
 			(hide yes)
@@
 			)
 		)
-		(property "MPN" "GRM21BR71H104KA01L"
+		(property "MPN" "C0805C104K5RACTU"
 			(at 330.2 228.6 0)
 			(hide yes)
@@
 			)
 		)
-		(property "Manufacturer" "Murata"
+		(property "Manufacturer" "KEMET"
 			(at 342.9 228.6 0)
 			(hide yes)
@@
 			)
 		)
-		(property "MPN" "GRM31MR71H105KA88L"
+		(property "MPN" "C1206C105K5RACTU"
 			(at 342.9 228.6 0)
 			(hide yes)
@@
 			)
 		)
-		(property "Manufacturer" "Yageo"
+		(property "Manufacturer" "Stackpole"
 			(at 370.84 129.54 0)
 			(hide yes)
@@
 			)
 		)
-		(property "MPN" "RC1206FR-07330RL"
+		(property "MPN" "RMCF1206FT330R"
 			(at 370.84 129.54 0)
 			(hide yes)
@@
 			)
 		)
-		(property "Manufacturer" "Yageo"
+		(property "Manufacturer" "Stackpole"
 			(at 370.84 152.4 0)
 			(hide yes)
@@
 			)
 		)
-		(property "MPN" "RC1206FR-07330RL"
+		(property "MPN" "RMCF1206FT330R"
 			(at 370.84 152.4 0)
 			(hide yes)
