File: boards/can-controller/hardware/ethernet.kicad_sch (KiCad schematic)
At the start: 37 parts, among them J4 JD0-0004NL, U3 W6100-L, Y2 25MHz

Commit message: Move core, can-card, io-card, serial-card, can-ssr, probe-helper to rev B
Rev A went to PCBWay and is tagged revA. Rev B replaces parts the Mouser
BOM check flagged (obsolete, end of life, not recommended for new designs,
or not orderable) and swaps out-of-stock passives and diodes for in-stock
equivalents. Field-only changes, same footprints, no layout change; the
reference boards (can-controller, pic-module) get the same part numbers.
The rev A order lists (DigiKey, Mouser) carry the same substitutions; the
Mouser list leaves out the T821 box headers (bought from DigiKey).

docs/rev-b-changes.md lists every change and the rev B to-dos (MAX7219 is
obsolete and must be replaced). transfer/mouser-revA.xlsx (Mouser BOM
check) consumed.

Co-Authored-By: Claude Opus 5.5 <noreply@anthropic.com>
Parts:
- C20, C21, C22, C23, C24, C25, C26, C27, C28, C32, C33, C34: MPN GRM21BR71H104KA01L -> C0805C104K5RACTU; Manufacturer Murata -> KEMET
- C35: MPN GRM31MR71H105KA88L -> C1206C105K5RACTU; Manufacturer Murata -> KEMET
- R22, R23: MPN RC1206FR-07330RL -> RMCF1206FT330R; Manufacturer Yageo -> Stackpole
Changed lines of the file:
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@@
 			)
 		)
-		(property "Manufacturer" "Murata"
+		(property "Manufacturer" "KEMET"
 			(at 127 55.88 0)
 			(hide yes)
@@
 			)
 		)
-		(property "MPN" "GRM21BR71H104KA01L"
+		(property "MPN" "C0805C104K5RACTU"
 			(at 127 55.88 0)
 			(hide yes)
@@
 			)
 		)
-		(property "Manufacturer" "Murata"
+		(property "Manufacturer" "KEMET"
 			(at 139.7 55.88 0)
 			(hide yes)
@@
 			)
 		)
-		(property "MPN" "GRM21BR71H104KA01L"
+		(property "MPN" "C0805C104K5RACTU"
 			(at 139.7 55.88 0)
 			(hide yes)
@@
 			)
 		)
-		(property "Manufacturer" "Murata"
+		(property "Manufacturer" "KEMET"
 			(at 152.4 55.88 0)
 			(hide yes)
@@
 			)
 		)
-		(property "MPN" "GRM21BR71H104KA01L"
+		(property "MPN" "C0805C104K5RACTU"
 			(at 152.4 55.88 0)
 			(hide yes)
@@
 			)
 		)
-		(property "Manufacturer" "Murata"
+		(property "Manufacturer" "KEMET"
 			(at 165.1 55.88 0)
 			(hide yes)
@@
 			)
 		)
-		(property "MPN" "GRM21BR71H104KA01L"
+		(property "MPN" "C0805C104K5RACTU"
 			(at 165.1 55.88 0)
 			(hide yes)
@@
 			)
 		)
-		(property "Manufacturer" "Murata"
+		(property "Manufacturer" "KEMET"
 			(at 177.8 55.88 0)
 			(hide yes)
@@
 			)
 		)
-		(property "MPN" "GRM21BR71H104KA01L"
+		(property "MPN" "C0805C104K5RACTU"
 			(at 177.8 55.88 0)
 			(hide yes)
@@
 			)
 		)
-		(property "Manufacturer" "Murata"
+		(property "Manufacturer" "KEMET"
 			(at 190.5 55.88 0)
 			(hide yes)
@@
 			)
 		)
-		(property "MPN" "GRM21BR71H104KA01L"
+		(property "MPN" "C0805C104K5RACTU"
 			(at 190.5 55.88 0)
 			(hide yes)
@@
 			)
 		)
-		(property "Manufacturer" "Murata"
+		(property "Manufacturer" "KEMET"
 			(at 203.2 55.88 0)
 			(hide yes)
@@
 			)
 		)
-		(property "MPN" "GRM21BR71H104KA01L"
+		(property "MPN" "C0805C104K5RACTU"
 			(at 203.2 55.88 0)
 			(hide yes)
@@
 			)
 		)
-		(property "Manufacturer" "Murata"
+		(property "Manufacturer" "KEMET"
 			(at 215.9 55.88 0)
 			(hide yes)
@@
 			)
 		)
-		(property "MPN" "GRM21BR71H104KA01L"
+		(property "MPN" "C0805C104K5RACTU"
 			(at 215.9 55.88 0)
 			(hide yes)
@@
 			)
 		)
-		(property "Manufacturer" "Murata"
+		(property "Manufacturer" "KEMET"
 			(at 228.6 55.88 0)
 			(hide yes)
@@
 			)
 		)
-		(property "MPN" "GRM21BR71H104KA01L"
+		(property "MPN" "C0805C104K5RACTU"
 			(at 228.6 55.88 0)
 			(hide yes)
@@
 			)
 		)
-		(property "Manufacturer" "Murata"
+		(property "Manufacturer" "KEMET"
 			(at 294.64 129.54 0)
 			(hide yes)
@@
 			)
 		)
-		(property "MPN" "GRM21BR71H104KA01L"
+		(property "MPN" "C0805C104K5RACTU"
 			(at 294.64 129.54 0)
 			(hide yes)
@@
 			)
 		)
-		(property "Manufacturer" "Murata"
+		(property "Manufacturer" "KEMET"
 			(at 294.64 172.72 0)
 			(hide yes)
@@
 			)
 		)
-		(property "MPN" "GRM21BR71H104KA01L"
+		(property "MPN" "C0805C104K5RACTU"
 			(at 294.64 172.72 0)
 			(hide yes)
@@
 			)
 		)
-		(property "Manufacturer" "Murata"
+		(property "Manufacturer" "KEMET"
 			(at 330.2 228.6 0)
 			(hide yes)
@@
 			)
 		)
-		(property "MPN" "GRM21BR71H104KA01L"
+		(property "MPN" "C0805C104K5RACTU"
 			(at 330.2 228.6 0)
 			(hide yes)
@@
 			)
 		)
-		(property "Manufacturer" "Murata"
+		(property "Manufacturer" "KEMET"
 			(at 342.9 228.6 0)
 			(hide yes)
@@
 			)
 		)
-		(property "MPN" "GRM31MR71H105KA88L"
+		(property "MPN" "C1206C105K5RACTU"
 			(at 342.9 228.6 0)
 			(hide yes)
@@
 			)
 		)
-		(property "Manufacturer" "Yageo"
+		(property "Manufacturer" "Stackpole"
 			(at 370.84 129.54 0)
 			(hide yes)
@@
 			)
 		)
-		(property "MPN" "RC1206FR-07330RL"
+		(property "MPN" "RMCF1206FT330R"
 			(at 370.84 129.54 0)
 			(hide yes)
@@
 			)
 		)
-		(property "Manufacturer" "Yageo"
+		(property "Manufacturer" "Stackpole"
 			(at 370.84 152.4 0)
 			(hide yes)
@@
 			)
 		)
-		(property "MPN" "RC1206FR-07330RL"
+		(property "MPN" "RMCF1206FT330R"
 			(at 370.84 152.4 0)
 			(hide yes)
