File: boards/can-controller/hardware/mcu.kicad_sch (KiCad schematic)
At the start: 26 parts, among them J2 ICSP, J3 UART, U1 PIC32MK1024MCM064-I/PT, U2 MCP1826S-3302E/DB, Y1 12MHz

Commit message: Move core, can-card, io-card, serial-card, can-ssr, probe-helper to rev B
Rev A went to PCBWay and is tagged revA. Rev B replaces parts the Mouser
BOM check flagged (obsolete, end of life, not recommended for new designs,
or not orderable) and swaps out-of-stock passives and diodes for in-stock
equivalents. Field-only changes, same footprints, no layout change; the
reference boards (can-controller, pic-module) get the same part numbers.
The rev A order lists (DigiKey, Mouser) carry the same substitutions; the
Mouser list leaves out the T821 box headers (bought from DigiKey).

docs/rev-b-changes.md lists every change and the rev B to-dos (MAX7219 is
obsolete and must be replaced). transfer/mouser-revA.xlsx (Mouser BOM
check) consumed.

Co-Authored-By: Claude Opus 5.5 <noreply@anthropic.com>
Parts:
- C1, C2, C8: MPN GRM31CR71E106KA12L -> CL31B106KAHNNNE; Manufacturer Murata -> Samsung Electro-Mechanics
- C10: MPN GRM31MR71H105KA88L -> C1206C105K5RACTU; Manufacturer Murata -> KEMET
- C11, C12: MPN GRM2165C1H270JA01D -> C0805C270J5GACTU; Manufacturer Murata -> KEMET
- C13, C3, C4, C5, C6, C7, C9: MPN GRM21BR71H104KA01L -> C0805C104K5RACTU; Manufacturer Murata -> KEMET
- D1, D2: MPN LTST-C150GKT -> LTST-C150KGKT
Changed lines of the file:
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@@
 			)
 		)
-		(property "Manufacturer" "Murata"
+		(property "Manufacturer" "Samsung Electro-Mechanics"
 			(at 45.72 76.2 0)
 			(hide yes)
@@
 			)
 		)
-		(property "MPN" "GRM31CR71E106KA12L"
+		(property "MPN" "CL31B106KAHNNNE"
 			(at 45.72 76.2 0)
 			(hide yes)
@@
 			)
 		)
-		(property "Manufacturer" "Murata"
+		(property "Manufacturer" "Samsung Electro-Mechanics"
 			(at 83.82 76.2 0)
 			(hide yes)
@@
 			)
 		)
-		(property "MPN" "GRM31CR71E106KA12L"
+		(property "MPN" "CL31B106KAHNNNE"
 			(at 83.82 76.2 0)
 			(hide yes)
@@
 			)
 		)
-		(property "MPN" "LTST-C150GKT"
+		(property "MPN" "LTST-C150KGKT"
 			(at 101.6 71.12 0)
 			(hide yes)
@@
 			)
 		)
-		(property "Manufacturer" "Murata"
+		(property "Manufacturer" "KEMET"
 			(at 152.4 45.72 0)
 			(hide yes)
@@
 			)
 		)
-		(property "MPN" "GRM21BR71H104KA01L"
+		(property "MPN" "C0805C104K5RACTU"
 			(at 152.4 45.72 0)
 			(hide yes)
@@
 			)
 		)
-		(property "Manufacturer" "Murata"
+		(property "Manufacturer" "KEMET"
 			(at 167.64 45.72 0)
 			(hide yes)
@@
 			)
 		)
-		(property "MPN" "GRM21BR71H104KA01L"
+		(property "MPN" "C0805C104K5RACTU"
 			(at 167.64 45.72 0)
 			(hide yes)
@@
 			)
 		)
-		(property "Manufacturer" "Murata"
+		(property "Manufacturer" "KEMET"
 			(at 182.88 45.72 0)
 			(hide yes)
@@
 			)
 		)
-		(property "MPN" "GRM21BR71H104KA01L"
+		(property "MPN" "C0805C104K5RACTU"
 			(at 182.88 45.72 0)
 			(hide yes)
@@
 			)
 		)
-		(property "Manufacturer" "Murata"
+		(property "Manufacturer" "KEMET"
 			(at 198.12 45.72 0)
 			(hide yes)
@@
 			)
 		)
-		(property "MPN" "GRM21BR71H104KA01L"
+		(property "MPN" "C0805C104K5RACTU"
 			(at 198.12 45.72 0)
 			(hide yes)
@@
 			)
 		)
-		(property "Manufacturer" "Murata"
+		(property "Manufacturer" "KEMET"
 			(at 213.36 45.72 0)
 			(hide yes)
@@
 			)
 		)
-		(property "MPN" "GRM21BR71H104KA01L"
+		(property "MPN" "C0805C104K5RACTU"
 			(at 213.36 45.72 0)
 			(hide yes)
@@
 			)
 		)
-		(property "Manufacturer" "Murata"
+		(property "Manufacturer" "Samsung Electro-Mechanics"
 			(at 228.6 45.72 0)
 			(hide yes)
@@
 			)
 		)
-		(property "MPN" "GRM31CR71E106KA12L"
+		(property "MPN" "CL31B106KAHNNNE"
 			(at 228.6 45.72 0)
 			(hide yes)
@@
 			)
 		)
-		(property "Manufacturer" "Murata"
+		(property "Manufacturer" "KEMET"
 			(at 116.84 129.54 0)
 			(hide yes)
@@
 			)
 		)
-		(property "MPN" "GRM21BR71H104KA01L"
+		(property "MPN" "C0805C104K5RACTU"
 			(at 116.84 129.54 0)
 			(hide yes)
@@
 			)
 		)
-		(property "Manufacturer" "Murata"
+		(property "Manufacturer" "KEMET"
 			(at 129.54 129.54 0)
 			(hide yes)
@@
 			)
 		)
-		(property "MPN" "GRM31MR71H105KA88L"
+		(property "MPN" "C1206C105K5RACTU"
 			(at 129.54 129.54 0)
 			(hide yes)
@@
 			)
 		)
-		(property "Manufacturer" "Murata"
+		(property "Manufacturer" "KEMET"
 			(at 335.28 129.54 0)
 			(hide yes)
@@
 			)
 		)
-		(property "MPN" "GRM2165C1H270JA01D"
+		(property "MPN" "C0805C270J5GACTU"
 			(at 335.28 129.54 0)
 			(hide yes)
@@
 			)
 		)
-		(property "Manufacturer" "Murata"
+		(property "Manufacturer" "KEMET"
 			(at 355.6 129.54 0)
 			(hide yes)
@@
 			)
 		)
-		(property "MPN" "GRM2165C1H270JA01D"
+		(property "MPN" "C0805C270J5GACTU"
 			(at 355.6 129.54 0)
 			(hide yes)
@@
 			)
 		)
-		(property "Manufacturer" "Murata"
+		(property "Manufacturer" "KEMET"
 			(at 76.2 175.26 0)
 			(hide yes)
@@
 			)
 		)
-		(property "MPN" "GRM21BR71H104KA01L"
+		(property "MPN" "C0805C104K5RACTU"
 			(at 76.2 175.26 0)
 			(hide yes)
@@
 			)
 		)
-		(property "MPN" "LTST-C150GKT"
+		(property "MPN" "LTST-C150KGKT"
 			(at 360.68 60.96 0)
 			(hide yes)

Commit message: Rev B / rev A order: 10 uF CL31B106KAHZW6E, beads BLM31PG391SN1L
Both earlier substitutes (CL31B106KAHNNNE, BLM31KN102SH1L) are on
backorder at Mouser. CL31B106KAHZW6E has the same rating (1.4 mm tall).
The isolated-supply beads need no 1 kOhm: TI's reference uses 330 Ohm;
BLM31PG391SN1L is 390 Ohm @ 100 MHz, 2 A, 50 mOhm. Field-only changes;
order lists regenerated.

Co-Authored-By: Claude Opus 5.5 <noreply@anthropic.com>
Parts:
- C1, C2, C8: MPN CL31B106KAHNNNE -> CL31B106KAHZW6E
Changed lines of the file:
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@@
 			)
 		)
-		(property "MPN" "CL31B106KAHNNNE"
+		(property "MPN" "CL31B106KAHZW6E"
 			(at 45.72 76.2 0)
 			(hide yes)
@@
 			)
 		)
-		(property "MPN" "CL31B106KAHNNNE"
+		(property "MPN" "CL31B106KAHZW6E"
 			(at 83.82 76.2 0)
 			(hide yes)
@@
 			)
 		)
-		(property "MPN" "CL31B106KAHNNNE"
+		(property "MPN" "CL31B106KAHZW6E"
 			(at 228.6 45.72 0)
 			(hide yes)
