File: boards/probe-helper/hardware/probe-helper.kicad_pcb (KiCad board)
At the start: 2 copper layers, 65 x 46 mm, 28 parts, among them J1 AD HAT terminal, J2 Pi pins 31-40, J3 PROBE A B

Commit message: Move core, can-card, io-card, serial-card, can-ssr, probe-helper to rev B
Rev A went to PCBWay and is tagged revA. Rev B replaces parts the Mouser
BOM check flagged (obsolete, end of life, not recommended for new designs,
or not orderable) and swaps out-of-stock passives and diodes for in-stock
equivalents. Field-only changes, same footprints, no layout change; the
reference boards (can-controller, pic-module) get the same part numbers.
The rev A order lists (DigiKey, Mouser) carry the same substitutions; the
Mouser list leaves out the T821 box headers (bought from DigiKey).

docs/rev-b-changes.md lists every change and the rev B to-dos (MAX7219 is
obsolete and must be replaced). transfer/mouser-revA.xlsx (Mouser BOM
check) consumed.

Co-Authored-By: Claude Opus 5.5 <noreply@anthropic.com>
Other:
- board text added: "PROBE HELPER rev B"
- board text removed: "PROBE HELPER rev A"
Changed lines of the file:
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@@
 		(title "Probe helper: ADS1263 HAT adapter")
 		(date "2026-10-11")
-		(rev "A")
+		(rev "B")
 	)
 	(layers
@@
 			)
 		)
-		(property "Manufacturer" "Sullins Connector Solutions"
+		(property "Manufacturer" "Amphenol FCI"
 			(at 0 0 180)
 			(layer "B.Fab")
@@
 			)
 		)
-		(property "MPN" "PRPC040SBAN-M71RC"
+		(property "MPN" "68016-136HLF"
 			(at 0 0 180)
 			(layer "B.Fab")
@@
 		)
 	)
-	(gr_text "PROBE HELPER rev A"
+	(gr_text "PROBE HELPER rev B"
 		(at 127.2 144.6 0)
 		(layer "F.SilkS")
