File: boards/probe-helper/hardware/probe-helper.kicad_sch (KiCad schematic)
At the start: 24 parts, among them J1 AD HAT terminal, J2 Pi pins 31-40, J3 PROBE A B

Commit message: probe-helper: 10M resistor MFR-25FBF52-10M (not orderable) -> Stackpole RNF14FTD10M0
Same 1/4 W axial body on the DIN0207 footprint; order list updated.

Co-Authored-By: Claude Opus 5.5 <noreply@anthropic.com>
Parts:
- R9: MPN MFR-25FBF52-10M -> RNF14FTD10M0; Manufacturer Yageo -> Stackpole
Changed lines of the file:
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@@
 			)
 		)
-		(property "Manufacturer" "Yageo"
+		(property "Manufacturer" "Stackpole"
 			(at 190.5 99.06 0)
 			(hide yes)
@@
 			)
 		)
-		(property "MPN" "MFR-25FBF52-10M"
+		(property "MPN" "RNF14FTD10M0"
 			(at 190.5 99.06 0)
 			(hide yes)

Commit message: Move core, can-card, io-card, serial-card, can-ssr, probe-helper to rev B
Rev A went to PCBWay and is tagged revA. Rev B replaces parts the Mouser
BOM check flagged (obsolete, end of life, not recommended for new designs,
or not orderable) and swaps out-of-stock passives and diodes for in-stock
equivalents. Field-only changes, same footprints, no layout change; the
reference boards (can-controller, pic-module) get the same part numbers.
The rev A order lists (DigiKey, Mouser) carry the same substitutions; the
Mouser list leaves out the T821 box headers (bought from DigiKey).

docs/rev-b-changes.md lists every change and the rev B to-dos (MAX7219 is
obsolete and must be replaced). transfer/mouser-revA.xlsx (Mouser BOM
check) consumed.

Co-Authored-By: Claude Opus 5.5 <noreply@anthropic.com>
Parts:
- J1: MPN PRPC040SBAN-M71RC -> 68016-136HLF; Manufacturer Sullins Connector Solutions -> Amphenol FCI
Changed lines of the file:
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@@
 		(title "Probe helper: ADS1263 HAT adapter")
 		(date "2026-10-11")
-		(rev "A")
+		(rev "B")
 	)
 	(text "Probe helper (docs/probe-helper-pi.md, tools/probe_ads1263.py). Plugs into the Waveshare High-Precision\nAD HAT's 13-way 3.5 mm screw terminal (J1) and takes 8 Pi GPIOs over a 10-way ribbon from the HAT's\npass-through header (J2). Each range is a GPIO divider: top GPIO high + bottom GPIO low puts its node\nN at 3.3 V x 47 / 1247 = 0.12 V behind ~45 R; both GPIOs as inputs (no pull) float it. The ADC reads\nN and both probe nodes; IDAC 1 mA out of IN3 (A) or IN1 (B) for the diode test."
@@
 			)
 		)
-		(property "Manufacturer" "Sullins Connector Solutions"
+		(property "Manufacturer" "Amphenol FCI"
 			(at 50.8 76.2 0)
 			(hide yes)
@@
 			)
 		)
-		(property "MPN" "PRPC040SBAN-M71RC"
+		(property "MPN" "68016-136HLF"
 			(at 50.8 76.2 0)
 			(hide yes)
