File: boards/io-card/hardware/io-card.kicad_sch (KiCad schematic)
At the start: 51 parts, among them J10 STACK BUS, J11 RACK 12V, J30 RELAY, J40 IO, K1 AQW212, K2 AQW212

Commit message: io-card: external relay drivers with 24 V coil option, MC terminals, placed + routed
Relay outputs drive external coils; JP1 selects rack +12 V or an external
coil supply (up to 24 V) on J30 9/10, fused by F30 1812L110/33MR; C70 50 V.
Terminals: SPTD double-level (24.2 mm) does not fit under the next card
(~11 mm), replaced by pluggable MC 1,5/10 and /12-G-3,5 (7.7 mm, FMC plugs),
signal next to return. J40 on the top edge (LOGIC), J30 on the bottom edge
(RACK); K1/K2 straddle a 2 mm copper-free gap. AI nets in net class HV
(0.8 mm). place.py / route.py (Freerouting); check_board clean.

Co-Authored-By: Claude Opus 5.5 <noreply@anthropic.com>
Parts:
- removed J30: RELAY, Thl_Connector:PhoenixContact_SPTD_1,5_4-H-3,5_2x04_P3.5mm_Horizontal, symbol Connector_Generic:Conn_02x04_Top_Bottom
- removed J40: IO, Thl_Connector:PhoenixContact_SPTD_1,5_6-H-3,5_2x06_P3.5mm_Horizontal, symbol Connector_Generic:Conn_02x06_Top_Bottom
- added J30: RELAY, Connector_Phoenix_MC:PhoenixContact_MC_1,5_10-G-3.5_1x10_P3.50mm_Horizontal, symbol Connector:Screw_Terminal_01x10
- added J40: IO, Connector_Phoenix_MC:PhoenixContact_MC_1,5_12-G-3.5_1x12_P3.50mm_Horizontal, symbol Connector:Screw_Terminal_01x12
- added JP1: COIL SUPPLY, Connector_PinHeader_2.54mm:PinHeader_1x03_P2.54mm_Vertical, symbol Jumper:Jumper_3_Open
- C70: value 10uF 25V X7R -> 4.7uF 50V X7R; MPN GRM31CR71E106KA12L -> GRM31CR71H475KA12L
- F30: value 1.1A -> 1.1A 33V; MPN 1812L110/16DR -> 1812L110/33MR
Connections:
- net +12V: now also JP1.1 (A); no longer F30.1
- net AIN1N: now also J40.10 (Pin_10)
- net AIN1P: now also J40.9 (Pin_9)
- net AIN2N: now also J40.12 (Pin_12)
- net AIN2P: now also J40.11 (Pin_11)
- net GND: now also J40.2 (Pin_2), J40.4 (Pin_4), J40.6 (Pin_6), J40.8 (Pin_8)
- net GND_RACK: now also J30.10 (Pin_10), J30.2 (Pin_2), J30.4 (Pin_4), J30.6 (Pin_6), J30.8 (Pin_8)
- net IO1: now also J40.1 (Pin_1)
- net IO2: now also J40.3 (Pin_3)
- net IO3: now also J40.5 (Pin_5)
- net IO4: now also J40.7 (Pin_7)
- net OUT1: now also J30.1 (Pin_1)
- net OUT2: now also J30.3 (Pin_3)
- net OUT3: now also J30.5 (Pin_5)
- net OUT4: now also J30.7 (Pin_7)
- net V12_RLY renamed V_RLY
- new net V_COIL_EXT: J30.9 (Pin_9), JP1.3 (B)
- new net V_COIL_SEL: F30.1, JP1.2 (C)
Other:
- note added: "J30 (MC 1,5/10-G-3,5 header, 7.7 mm: fits under the next card; plug FMC 1,5/10-ST-3,5 push-in): 1/2 OUT1 / 0 V, 3/4 OUT2 / 0 V, 5/6 OUT3 / 0 V, 7/8 OUT4 / 0 V (OUTn = coil +, V_RLY when on), 9/10 external coil supply + / 0 V (0 V = GND_RACK). Coils up to about 100 mA each; F30 1.1 A hold for all four. LEDs: 2 mA at 12 V, 4.7 mA at 24 V."
- note added: "J40 (MC 1,5/12-G-3,5, plug FMC 1,5/12-ST-3,5): 1/2 IO1 / GND, 3/4 IO2 / GND, 5/6 IO3 / GND, 7/8 IO4 / GND, 9/10 AI1+ / AI1-, 11/12 AI2+ / AI2-."
- note added: "RELAY DRIVE (requirements 4.1): four drivers for EXTERNAL relay coils. 2 x AQW212 PhotoMOS (2 Form A, 60 V, 0.5 A, 2.5 R max per channel). LED side LOGIC: RLYn (core PIC32 pin, 3.3 V) -> 470R -> LED -> GND, (3.3 - 1.5 V) / 470R >= 3.8 mA against 3 mA max operate. Output side RACK: V_RLY -> contact -> OUTn; the coil returns to GND_RACK on the same terminal pair. Coil supply by JP1: 1-2 rack +12V (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"
- note removed: "J30 (SPTD 1,5/4-H-3,5, double-level push-in): lower level 1-4 = OUT1-4 (+12 V when on), upper level 5-8 = 0 V (GND_RACK). Coils up to about 100 mA each; F30 1.1 A hold for all four."
- note removed: "J40 (SPTD 1,5/6-H-3,5): lower level 1-4 IO1-4, 5 AI1+, 6 AI2+; upper level 7-10 GND (one per GPIO), 11 AI1-, 12 AI2-."
- note removed: "RELAY DRIVE (requirements 4.1): four outputs for standard 12 V coil relays. 2 x AQW212 PhotoMOS (2 Form A, 60 V, 0.5 A, 2.5 R max per channel). LED side LOGIC: RLYn (core PIC32 pin, 3.3 V) -> 470R -> LED -> GND, (3.3 - 1.5 V) / 470R >= 3.8 mA against 3 mA max operate. Output side RACK: +12V (J11, after the core's input protection) -> F30 -> V12_RLY -> contact -> OUTn; the coil returns to GND_RACK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"

Commit message: io-card VMID isolation (R88 1k + C85 100 nF); relay failsafe timeout (core fw 0.4)
io-card: VMID from the core's OA5 (rated for 32 pF) now reaches the AI
dividers through R88 1k + C85 100 nF to GND (VMID_F). Rerouted, check_board
clean; AQW212 GND pins solid to the pours (starved thermal).

core: RLY takes an optional timeout=<ms> (100-3600000) for the outputs it
names; an output on with a timeout switches off unless an RLY naming it
arrives in time, and is reported in expired= until commanded again. No
timeout = no failsafe. A bare RLY does not restart timers.

Co-Authored-By: Claude Opus 5.5 <noreply@anthropic.com>
Parts:
- added C85: 100nF 50V X7R, Capacitor_SMD:C_0805_2012Metric_Pad1.18x1.45mm_HandSolder, symbol Device:C
- added R88: 1k, Resistor_SMD:R_1206_3216Metric_Pad1.30x1.75mm_HandSolder, symbol Device:R
Connections:
- net GND: now also C85.2
- net VMID: now also R88.1; no longer C80.2, C81.2, C82.2, C83.2, R84.2, R85.2, R86.2, R87.2
- new net VMID_F: C80.2, C81.2, C82.2, C83.2, C85.1, R84.2, R85.2, R86.2, R87.2, R88.2

Commit message: io-card: 4 x 0-10 V analog outputs; core fw 0.5 AO command
Hardware (boards/io-card):
- RACK-domain analog out from rack +12 V, 0 V = GND_RACK shared by all four
  and the relay returns: I2C1 -> ISO1540 -> MCP4728 (0x60, 2.048 V x 2) ->
  OPA4171 x 2.5 (10.24 V FS), 47R inside the loop + 1 nF, BAT54S clamps,
  MC78L05 for the 5 V side; J50 MC 1,5/8 on the right edge.
- Top-right corner becomes RACK (gap at x 61.5, U90 straddles it).
- Schematic sheet A2 (AO band below the original A3 area).
- Routed onto the reviewed board with route.py ao: existing tracks locked
  and returned unchanged; DAC fan-out pre-routed (net class Fine, MSOP
  pad-spacing DRC rule); Freerouting fragments on routed nets removed.
- check_board clean (ERC, DRC + schematic parity).

Firmware (boards/core): i2c.c (polled I2C1 master, bus recovery), AO
command with RLY-style optional failsafe to 0 V, ao= in IO/STATUS.
Not yet run on hardware.

Docs: requirements (core + cards is the final product; AO back on the
io-card), PROTOCOL.md, READMEs. Tools: schgen multi-unit symbols and
junctions, miniroute ground_fanout refs filter. Lib: LM2902, MC78L05_SOT89,
ISO1540, MCP4728 (+ MSOP-10, SOT-89-3).

Co-Authored-By: Claude Opus 5.5 <noreply@anthropic.com>
Parts:
- added C90, C91, C92, C94, C95: 100nF 50V X7R, Capacitor_SMD:C_0805_2012Metric_Pad1.18x1.45mm_HandSolder, symbol Device:C
- added C93: 10uF 25V X7R, Capacitor_SMD:C_1206_3216Metric_Pad1.33x1.80mm_HandSolder, symbol Device:C
- added C96, C97, C98, C99: 1nF 50V C0G, Capacitor_SMD:C_1206_3216Metric_Pad1.33x1.80mm_HandSolder, symbol Device:C
- added D90, D91, D92, D93: BAT54S, Package_TO_SOT_SMD:SOT-23, symbol Diode:BAT54S
- added J50: ANALOG OUT, Connector_Phoenix_MC:PhoenixContact_MC_1,5_8-G-3.5_1x08_P3.50mm_Horizontal, symbol Connector:Screw_Terminal_01x08
- added R100, R101, R102, R103: 47R, Resistor_SMD:R_1206_3216Metric_Pad1.30x1.75mm_HandSolder, symbol Device:R
- added R90, R91: 4.7k, Resistor_SMD:R_1206_3216Metric_Pad1.30x1.75mm_HandSolder, symbol Device:R
- added R92, R93, R94, R95: 10k 0.1%, Resistor_SMD:R_1206_3216Metric_Pad1.30x1.75mm_HandSolder, symbol Device:R
- added R96, R97, R98, R99: 15k 0.1%, Resistor_SMD:R_1206_3216Metric_Pad1.30x1.75mm_HandSolder, symbol Device:R
- added U90: ISO1540, Package_SO:SOIC-8_3.9x4.9mm_P1.27mm, symbol Isolator:ISO1540
- added U91: MC78L05, Package_TO_SOT_SMD:SOT-89-3, symbol Regulator_Linear:MC78L05_SOT89
- added U92: MCP4728, Package_SO:MSOP-10_3x3mm_P0.5mm, symbol Analog_DAC:MCP4728
- added U93: OPA4171, Package_SO:SOIC-14_3.9x8.7mm_P1.27mm, symbol Amplifier_Operational:LM2902
Connections:
- net +12V: now also C92.1, C95.1, D90.2 (K), D91.2 (K), D92.2 (K), D93.2 (K), U91.3 (IN), U93.4 (V+)
- net +3V3: now also C90.1, U90.1 (VCC1)
- net GND: now also C90.2, U90.4 (GND1)
- net GND_RACK: now also C91.2, C92.2, C93.2, C94.2, C95.2, D90.1 (A), D91.1 (A), D92.1 (A), D93.1 (A), J50.2 (Pin_2), J50.4 (Pin_4), J50.6 (Pin_6), J50.8 (Pin_8), R92.2, R93.2, R94.2, R95.2, U90.5 (GND2), U91.2 (GND), U92.10 (VSS), U92.4 (~{LDAC}), U93.11 (V-)
- net SDA: now reaches J10.15 (Pin_15)
- net SDA: now also U90.2 (SDA1)
- net SCL: now reaches J10.16 (Pin_16)
- net SCL: now also U90.3 (SCL1)
- new net: C98.1, R94.1, R98.1, U93.9 (-)
- new net: C99.1, R95.1, R99.1, U93.13 (-)
- new net: C99.2, R103.1, U93.14
- new net: C97.2, R101.1, U93.7
- new net: C96.1, R92.1, R96.1, U93.2 (-)
- new net: C97.1, R93.1, R97.1, U93.6 (-)
- new net: C96.2, R100.1, U93.1
- new net: C98.2, R102.1, U93.8
- new net AO1: D90.3 (COM), J50.1 (Pin_1), R100.2, R96.2
- new net AO2: D91.3 (COM), J50.3 (Pin_3), R101.2, R97.2
- new net AO3: D92.3 (COM), J50.5 (Pin_5), R102.2, R98.2
- new net AO4: D93.3 (COM), J50.7 (Pin_7), R103.2, R99.2
- new net AO_SCL: R91.2, U90.6 (SCL2), U92.2 (SCL)
- new net AO_SDA: R90.2, U90.7 (SDA2), U92.3 (SDA)
- new net DAC1: U92.6 (VOUTA), U93.3 (+)
- new net DAC2: U92.7 (VOUTB), U93.5 (+)
- new net DAC3: U92.8 (VOUTC), U93.10 (+)
- new net DAC4: U92.9 (VOUTD), U93.12 (+)
- new net V5_AO: C91.1, C93.1, C94.1, R90.1, R91.1, U90.8 (VCC2), U91.1 (OUT), U92.1 (VDD)
- no-connect marks 20 -> 19
Other:
- note added: "ANALOG OUT: four 0-10 V outputs, 10 mA each, in the RACK domain: powered from rack +12V, 0 V = GND_RACK (the relay 0 V; all outputs share it). I2C1 from the stack bus crosses through U90 (ISO1540, 2500 Vrms, the core's 4.7k pull-ups on side 1; its side-1 low is up to 0.8 V, so no other ISO15xx side 1 on the bus). U92 MCP4728 at 0x60 (address bits 000), internal 2.048 V reference x 2 = 4.096 V, ~L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"
- note added: "J50 (MC 1,5/8-G-3,5, plug FMC 1,5/8-ST-3,5): 1/2 AO1 / 0 V, 3/4 AO2 / 0 V, 5/6 AO3 / 0 V, 7/8 AO4 / 0 V (0 V = GND_RACK)."
- title: IO card: relays, GPIO, differential AI -> IO card: relays, GPIO, differential AI, analog out

Commit message: io-card: U92 MSOP-10 pads narrowed to 0.30 mm for PCBWay's mask web
PCBWay (order W517176ASE106) needs >= 0.19 mm between IC pads for a green
solder-mask web; the stock MSOP-10 pads (0.35 mm) left 0.15 mm. New
Thl_Package:MSOP-10_3x3mm_P0.5mm_Pad0.30 (stock footprint, 0.30 mm pads
per Microchip's MSOP-10 UN land pattern, 0.20 mm gap), built by
lib/footprint_src/Thl_Package/msop10_pad030.py. U92 tracks (0.20/0.25 mm)
still land inside the pads; check_board clean. No other pad gap under
0.19 mm on the six ordered boards.

Co-Authored-By: Claude Opus 5.5 <noreply@anthropic.com>
Parts:
- U92: footprint Package_SO:MSOP-10_3x3mm_P0.5mm -> Thl_Package:MSOP-10_3x3mm_P0.5mm_Pad0.30
Changed lines of the file:
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@@
 			)
 		)
-		(property "Footprint" "Package_SO:MSOP-10_3x3mm_P0.5mm"
+		(property "Footprint" "Thl_Package:MSOP-10_3x3mm_P0.5mm_Pad0.30"
 			(at 129.54 350.52 0)
 			(hide yes)

Commit message: Move core, can-card, io-card, serial-card, can-ssr, probe-helper to rev B
Rev A went to PCBWay and is tagged revA. Rev B replaces parts the Mouser
BOM check flagged (obsolete, end of life, not recommended for new designs,
or not orderable) and swaps out-of-stock passives and diodes for in-stock
equivalents. Field-only changes, same footprints, no layout change; the
reference boards (can-controller, pic-module) get the same part numbers.
The rev A order lists (DigiKey, Mouser) carry the same substitutions; the
Mouser list leaves out the T821 box headers (bought from DigiKey).

docs/rev-b-changes.md lists every change and the rev B to-dos (MAX7219 is
obsolete and must be replaced). transfer/mouser-revA.xlsx (Mouser BOM
check) consumed.

Co-Authored-By: Claude Opus 5.5 <noreply@anthropic.com>
Parts:
- C1, C85, C90, C91, C92, C94, C95: MPN GRM21BR71H104KA01L -> C0805C104K5RACTU; Manufacturer Murata -> KEMET
- C2, C71, C93: MPN GRM31CR71E106KA12L -> CL31B106KAHNNNE; Manufacturer Murata -> Samsung Electro-Mechanics
- C70: MPN GRM31CR71H475KA12L -> CL31B475KBHNNNE; Manufacturer Murata -> Samsung Electro-Mechanics
- C80, C81, C82, C83: MPN GRM319R71H104KA01D -> C1206C104K5RACTU; Manufacturer Murata -> KEMET
- C96, C97, C98, C99: MPN GRM3195C1H102JA01D -> C1206C102J5GACTU; Manufacturer Murata -> KEMET
- D51, D52, D53, D54, D55, D56, D57, D58, D90, D91, D92, D93: MPN BAT54S,215 -> BAT54S-7-F; Manufacturer Nexperia -> Diodes Incorporated
- R71, R72, R73, R74: MPN RC1206FR-07330RL -> RMCF1206FT330R; Manufacturer Yageo -> Stackpole

Commit message: Rev B / rev A order: 10 uF CL31B106KAHZW6E, beads BLM31PG391SN1L
Both earlier substitutes (CL31B106KAHNNNE, BLM31KN102SH1L) are on
backorder at Mouser. CL31B106KAHZW6E has the same rating (1.4 mm tall).
The isolated-supply beads need no 1 kOhm: TI's reference uses 330 Ohm;
BLM31PG391SN1L is 390 Ohm @ 100 MHz, 2 A, 50 mOhm. Field-only changes;
order lists regenerated.

Co-Authored-By: Claude Opus 5.5 <noreply@anthropic.com>
Parts:
- C2, C71, C93: MPN CL31B106KAHNNNE -> CL31B106KAHZW6E
Changed lines of the file:
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@@
 			)
 		)
-		(property "MPN" "CL31B106KAHNNNE"
+		(property "MPN" "CL31B106KAHZW6E"
 			(at 96.52 76.2 0)
 			(hide yes)
@@
 			)
 		)
-		(property "MPN" "CL31B106KAHNNNE"
+		(property "MPN" "CL31B106KAHZW6E"
 			(at 66.04 391.16 0)
 			(hide yes)
@@
 			)
 		)
-		(property "MPN" "CL31B106KAHNNNE"
+		(property "MPN" "CL31B106KAHZW6E"
 			(at 363.22 190.5 0)
 			(hide yes)
