File: boards/serial-card/hardware/serial-card.kicad_pcb (KiCad board)
At the start: 2 copper layers, 100 x 100 mm, 102 parts, among them J10 STACK BUS, J11 RACK 12V, J20 RS-232 1, J21 RS-232 2, J30 RS-485 3, J31 RS-485 4, U1 ST3232B, U10 ISOW1432, U11 ISOW1432

Commit message: Move core, can-card, io-card, serial-card, can-ssr, probe-helper to rev B
Rev A went to PCBWay and is tagged revA. Rev B replaces parts the Mouser
BOM check flagged (obsolete, end of life, not recommended for new designs,
or not orderable) and swaps out-of-stock passives and diodes for in-stock
equivalents. Field-only changes, same footprints, no layout change; the
reference boards (can-controller, pic-module) get the same part numbers.
The rev A order lists (DigiKey, Mouser) carry the same substitutions; the
Mouser list leaves out the T821 box headers (bought from DigiKey).

docs/rev-b-changes.md lists every change and the rev B to-dos (MAX7219 is
obsolete and must be replaced). transfer/mouser-revA.xlsx (Mouser BOM
check) consumed.

Co-Authored-By: Claude Opus 5.5 <noreply@anthropic.com>
Parts:
- FB10, FB11, FB12, FB13: value BLM31KN102SN1L -> BLM31KN102SH1L
Changed lines of the file:
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@@
 		(title "Serial card: 2 x RS-232, 2 x isolated RS-485")
 		(date "2026-10-09")
-		(rev "A")
+		(rev "B")
 	)
 	(layers
@@
 			)
 		)
-		(property "MPN" "LTST-C150GKT"
+		(property "MPN" "LTST-C150KGKT"
 			(at 0 0 0)
 			(layer "F.Fab")
@@
 			)
 		)
-		(property "Manufacturer" "Murata"
+		(property "Manufacturer" "KEMET"
 			(at 0 0 90)
 			(layer "F.Fab")
@@
 			)
 		)
-		(property "MPN" "GRM319R71H104KA01D"
+		(property "MPN" "C1206C104K5RACTU"
 			(at 0 0 90)
 			(layer "F.Fab")
@@
 			)
 		)
-		(property "Manufacturer" "Murata"
+		(property "Manufacturer" "KEMET"
 			(at 0 0 90)
 			(layer "F.Fab")
@@
 			)
 		)
-		(property "MPN" "GRM21BR71H104KA01L"
+		(property "MPN" "C0805C104K5RACTU"
 			(at 0 0 90)
 			(layer "F.Fab")
@@
 			)
 		)
-		(property "Manufacturer" "Murata"
+		(property "Manufacturer" "KEMET"
 			(at 0 0 270)
 			(layer "F.Fab")
@@
 			)
 		)
-		(property "MPN" "GRM21BR71H103KA01L"
+		(property "MPN" "C0805C103K5RACTU"
 			(at 0 0 270)
 			(layer "F.Fab")
@@
 			)
 		)
-		(property "Value" "BLM31KN102SN1L"
+		(property "Value" "BLM31KN102SH1L"
 			(at 0 1.9 0)
 			(layer "F.Fab")
@@
 			)
 		)
-		(property "MPN" "BLM31KN102SN1L"
+		(property "MPN" "BLM31KN102SH1L"
 			(at 0 0 0)
 			(layer "F.Fab")
@@
 			)
 		)
-		(property "Manufacturer" "Murata"
+		(property "Manufacturer" "KEMET"
 			(at 0 0 90)
 			(layer "F.Fab")
@@
 			)
 		)
-		(property "MPN" "GRM21BR71H104KA01L"
+		(property "MPN" "C0805C104K5RACTU"
 			(at 0 0 90)
 			(layer "F.Fab")
@@
 			)
 		)
-		(property "Manufacturer" "Murata"
+		(property "Manufacturer" "KEMET"
 			(at 0 0 270)
 			(layer "F.Fab")
@@
 			)
 		)
-		(property "MPN" "GRM31MR71H105KA88L"
+		(property "MPN" "C1206C105K5RACTU"
 			(at 0 0 270)
 			(layer "F.Fab")
@@
 			)
 		)
-		(property "Manufacturer" "Murata"
+		(property "Manufacturer" "KEMET"
 			(at 0 0 270)
 			(layer "F.Fab")
@@
 			)
 		)
-		(property "MPN" "GRM31MR71H105KA88L"
+		(property "MPN" "C1206C105K5RACTU"
 			(at 0 0 270)
 			(layer "F.Fab")
@@
 			)
 		)
-		(property "Manufacturer" "Murata"
+		(property "Manufacturer" "Samsung Electro-Mechanics"
 			(at 0 0 270)
 			(layer "F.Fab")
@@
 			)
 		)
-		(property "MPN" "GRM31CR71E106KA12L"
+		(property "MPN" "CL31B106KAHNNNE"
 			(at 0 0 270)
 			(layer "F.Fab")
@@
 			)
 		)
-		(property "Manufacturer" "Murata"
+		(property "Manufacturer" "KEMET"
 			(at 0 0 90)
 			(layer "F.Fab")
@@
 			)
 		)
-		(property "MPN" "GRM21BR71H104KA01L"
+		(property "MPN" "C0805C104K5RACTU"
 			(at 0 0 90)
 			(layer "F.Fab")
@@
 			)
 		)
-		(property "Manufacturer" "Murata"
+		(property "Manufacturer" "KEMET"
 			(at 0 0 270)
 			(layer "F.Fab")
@@
 			)
 		)
-		(property "MPN" "GRM31MR71H105KA88L"
+		(property "MPN" "C1206C105K5RACTU"
 			(at 0 0 270)
 			(layer "F.Fab")
@@
 			)
 		)
-		(property "Value" "BLM31KN102SN1L"
+		(property "Value" "BLM31KN102SH1L"
 			(at 0 1.9 0)
 			(layer "F.Fab")
@@
 			)
 		)
-		(property "MPN" "BLM31KN102SN1L"
+		(property "MPN" "BLM31KN102SH1L"
 			(at 0 0 0)
 			(layer "F.Fab")
@@
 			)
 		)
-		(property "Manufacturer" "Murata"
+		(property "Manufacturer" "KEMET"
 			(at 0 0 0)
 			(layer "F.Fab")
@@
 			)
 		)
-		(property "MPN" "GRM319R71H104KA01D"
+		(property "MPN" "C1206C104K5RACTU"
 			(at 0 0 0)
 			(layer "F.Fab")
@@
 			)
 		)
-		(property "MPN" "LTST-C150GKT"
+		(property "MPN" "LTST-C150KGKT"
 			(at 0 0 0)
 			(layer "F.Fab")
@@
 			)
 		)
-		(property "Value" "BLM31KN102SN1L"
+		(property "Value" "BLM31KN102SH1L"
 			(at 0 1.9 90)
 			(layer "F.Fab")
@@
 			)
 		)
-		(property "MPN" "BLM31KN102SN1L"
+		(property "MPN" "BLM31KN102SH1L"
 			(at 0 0 90)
 			(layer "F.Fab")
@@
 			)
 		)
-		(property "Manufacturer" "Murata"
+		(property "Manufacturer" "Samsung Electro-Mechanics"
 			(at 0 0 0)
 			(layer "F.Fab")
@@
 			)
 		)
-		(property "MPN" "GRM31CR71E106KA12L"
+		(property "MPN" "CL31B106KAHNNNE"
 			(at 0 0 0)
 			(layer "F.Fab")
@@
 			)
 		)
-		(property "Manufacturer" "Murata"
+		(property "Manufacturer" "Samsung Electro-Mechanics"
 			(at 0 0 270)
 			(layer "F.Fab")
@@
 			)
 		)
-		(property "MPN" "GRM31CR71E106KA12L"
+		(property "MPN" "CL31B106KAHNNNE"
 			(at 0 0 270)
 			(layer "F.Fab")
@@
 			)
 		)
-		(property "MPN" "LTST-C150GKT"
+		(property "MPN" "LTST-C150KGKT"
 			(at 0 0 0)
 			(layer "F.Fab")
@@
 			)
 		)
-		(property "Manufacturer" "Murata"
+		(property "Manufacturer" "KEMET"
 			(at 0 0 0)
 			(layer "F.Fab")
@@
 			)
 		)
-		(property "MPN" "GRM319R71H104KA01D"
+		(property "MPN" "C1206C104K5RACTU"
 			(at 0 0 0)
 			(layer "F.Fab")
@@
 			)
 		)
-		(property "Manufacturer" "Murata"
+		(property "Manufacturer" "KEMET"
 			(at 0 0 270)
 			(layer "F.Fab")
@@
 			)
 		)
-		(property "MPN" "GRM21BR71H103KA01L"
+		(property "MPN" "C0805C103K5RACTU"
 			(at 0 0 270)
 			(layer "F.Fab")
@@
 			)
 		)
-		(property "Manufacturer" "Murata"
+		(property "Manufacturer" "Samsung Electro-Mechanics"
 			(at 0 0 90)
 			(layer "F.Fab")
@@
 			)
 		)
-		(property "MPN" "GRM31CR71E106KA12L"
+		(property "MPN" "CL31B106KAHNNNE"
 			(at 0 0 90)
 			(layer "F.Fab")
@@
 			)
 		)
-		(property "Manufacturer" "Murata"
+		(property "Manufacturer" "Samsung Electro-Mechanics"
 			(at 0 0 90)
 			(layer "F.Fab")
@@
 			)
 		)
-		(property "MPN" "GRM31CR71E106KA12L"
+		(property "MPN" "CL31B106KAHNNNE"
 			(at 0 0 90)
 			(layer "F.Fab")
@@
 			)
 		)
-		(property "Value" "BLM31KN102SN1L"
+		(property "Value" "BLM31KN102SH1L"
 			(at 0 1.9 90)
 			(layer "F.Fab")
@@
 			)
 		)
-		(property "MPN" "BLM31KN102SN1L"
+		(property "MPN" "BLM31KN102SH1L"
 			(at 0 0 90)
 			(layer "F.Fab")
@@
 			)
 		)
-		(property "MPN" "LTST-C150GKT"
+		(property "MPN" "LTST-C150KGKT"
 			(at 0 0 0)
 			(layer "F.Fab")
@@
 			)
 		)
-		(property "Manufacturer" "Murata"
+		(property "Manufacturer" "KEMET"
 			(at 0 0 270)
 			(layer "F.Fab")
@@
 			)
 		)
-		(property "MPN" "GRM21BR71H103KA01L"
+		(property "MPN" "C0805C103K5RACTU"
 			(at 0 0 270)
 			(layer "F.Fab")
@@
 			)
 		)
-		(property "Manufacturer" "Murata"
+		(property "Manufacturer" "Samsung Electro-Mechanics"
 			(at 0 0 0)
 			(layer "F.Fab")
@@
 			)
 		)
-		(property "MPN" "GRM31CR71E106KA12L"
+		(property "MPN" "CL31B106KAHNNNE"
 			(at 0 0 0)
 			(layer "F.Fab")
@@
 			)
 		)
-		(property "Manufacturer" "Murata"
+		(property "Manufacturer" "Samsung Electro-Mechanics"
 			(at 0 0 270)
 			(layer "F.Fab")
@@
 			)
 		)
-		(property "MPN" "GRM31CR71E106KA12L"
+		(property "MPN" "CL31B106KAHNNNE"
 			(at 0 0 270)
 			(layer "F.Fab")
@@
 			)
 		)
-		(property "Manufacturer" "Murata"
+		(property "Manufacturer" "KEMET"
 			(at 0 0 90)
 			(layer "F.Fab")
@@
 			)
 		)
-		(property "MPN" "GRM21BR71H104KA01L"
+		(property "MPN" "C0805C104K5RACTU"
 			(at 0 0 90)
 			(layer "F.Fab")
@@
 			)
 		)
-		(property "Manufacturer" "Murata"
+		(property "Manufacturer" "Samsung Electro-Mechanics"
 			(at 0 0 270)
 			(layer "F.Fab")
@@
 			)
 		)
-		(property "MPN" "GRM31CR71E106KA12L"
+		(property "MPN" "CL31B106KAHNNNE"
 			(at 0 0 270)
 			(layer "F.Fab")
@@
 			)
 		)
-		(property "Manufacturer" "Murata"
+		(property "Manufacturer" "KEMET"
 			(at 0 0 90)
 			(layer "F.Fab")
@@
 			)
 		)
-		(property "MPN" "GRM319R71H104KA01D"
+		(property "MPN" "C1206C104K5RACTU"
 			(at 0 0 90)
 			(layer "F.Fab")
@@
 			)
 		)
-		(property "Manufacturer" "Murata"
+		(property "Manufacturer" "KEMET"
 			(at 0 0 90)
 			(layer "F.Fab")
@@
 			)
 		)
-		(property "MPN" "GRM21BR71H104KA01L"
+		(property "MPN" "C0805C104K5RACTU"
 			(at 0 0 90)
 			(layer "F.Fab")
@@
 			)
 		)
-		(property "Manufacturer" "Murata"
+		(property "Manufacturer" "KEMET"
 			(at 0 0 270)
 			(layer "F.Fab")
@@
 			)
 		)
-		(property "MPN" "GRM31MR71H105KA88L"
+		(property "MPN" "C1206C105K5RACTU"
 			(at 0 0 270)
 			(layer "F.Fab")
@@
 			)
 		)
-		(property "Manufacturer" "Murata"
+		(property "Manufacturer" "KEMET"
 			(at 0 0 270)
 			(layer "F.Fab")
@@
 			)
 		)
-		(property "MPN" "GRM21BR71H103KA01L"
+		(property "MPN" "C0805C103K5RACTU"
 			(at 0 0 270)
 			(layer "F.Fab")

Commit message: Rev B / rev A order: 10 uF CL31B106KAHZW6E, beads BLM31PG391SN1L
Both earlier substitutes (CL31B106KAHNNNE, BLM31KN102SH1L) are on
backorder at Mouser. CL31B106KAHZW6E has the same rating (1.4 mm tall).
The isolated-supply beads need no 1 kOhm: TI's reference uses 330 Ohm;
BLM31PG391SN1L is 390 Ohm @ 100 MHz, 2 A, 50 mOhm. Field-only changes;
order lists regenerated.

Co-Authored-By: Claude Opus 5.5 <noreply@anthropic.com>
Parts:
- FB10, FB11, FB12, FB13: value BLM31KN102SH1L -> BLM31PG391SN1L
Changed lines of the file:
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@@
 			)
 		)
-		(property "Value" "BLM31KN102SH1L"
+		(property "Value" "BLM31PG391SN1L"
 			(at 0 1.9 0)
 			(layer "F.Fab")
@@
 			)
 		)
-		(property "MPN" "BLM31KN102SH1L"
+		(property "MPN" "BLM31PG391SN1L"
 			(at 0 0 0)
 			(layer "F.Fab")
@@
 			)
 		)
-		(property "MPN" "CL31B106KAHNNNE"
+		(property "MPN" "CL31B106KAHZW6E"
 			(at 0 0 270)
 			(layer "F.Fab")
@@
 			)
 		)
-		(property "Value" "BLM31KN102SH1L"
+		(property "Value" "BLM31PG391SN1L"
 			(at 0 1.9 0)
 			(layer "F.Fab")
@@
 			)
 		)
-		(property "MPN" "BLM31KN102SH1L"
+		(property "MPN" "BLM31PG391SN1L"
 			(at 0 0 0)
 			(layer "F.Fab")
@@
 			)
 		)
-		(property "Value" "BLM31KN102SH1L"
+		(property "Value" "BLM31PG391SN1L"
 			(at 0 1.9 90)
 			(layer "F.Fab")
@@
 			)
 		)
-		(property "MPN" "BLM31KN102SH1L"
+		(property "MPN" "BLM31PG391SN1L"
 			(at 0 0 90)
 			(layer "F.Fab")
@@
 			)
 		)
-		(property "MPN" "CL31B106KAHNNNE"
+		(property "MPN" "CL31B106KAHZW6E"
 			(at 0 0 0)
 			(layer "F.Fab")
@@
 			)
 		)
-		(property "MPN" "CL31B106KAHNNNE"
+		(property "MPN" "CL31B106KAHZW6E"
 			(at 0 0 270)
 			(layer "F.Fab")
@@
 			)
 		)
-		(property "MPN" "CL31B106KAHNNNE"
+		(property "MPN" "CL31B106KAHZW6E"
 			(at 0 0 90)
 			(layer "F.Fab")
@@
 			)
 		)
-		(property "MPN" "CL31B106KAHNNNE"
+		(property "MPN" "CL31B106KAHZW6E"
 			(at 0 0 90)
 			(layer "F.Fab")
@@
 			)
 		)
-		(property "Value" "BLM31KN102SH1L"
+		(property "Value" "BLM31PG391SN1L"
 			(at 0 1.9 90)
 			(layer "F.Fab")
@@
 			)
 		)
-		(property "MPN" "BLM31KN102SH1L"
+		(property "MPN" "BLM31PG391SN1L"
 			(at 0 0 90)
 			(layer "F.Fab")
@@
 			)
 		)
-		(property "MPN" "CL31B106KAHNNNE"
+		(property "MPN" "CL31B106KAHZW6E"
 			(at 0 0 0)
 			(layer "F.Fab")
@@
 			)
 		)
-		(property "MPN" "CL31B106KAHNNNE"
+		(property "MPN" "CL31B106KAHZW6E"
 			(at 0 0 270)
 			(layer "F.Fab")
@@
 			)
 		)
-		(property "MPN" "CL31B106KAHNNNE"
+		(property "MPN" "CL31B106KAHZW6E"
 			(at 0 0 270)
 			(layer "F.Fab")
