File: boards/can-card/hardware/can-card.kicad_pcb (KiCad board)
At the start: 2 copper layers, 100 x 100 mm, 81 parts, among them J10 STACK BUS, J11 RACK 12V, J21 CAN1, J22 CAN2, J23 CAN3, J24 CAN4, U10 ISOW1044, U11 ISOW1044, U12 ISOW1044, U13 ISOW1044

Commit message: Probe test points on all fab boards; golden-board R/C/L test tool
tools/testpoints.py puts a 1.0 mm bare-copper pad (Thl_TestPoint:
TP_Probe_D1.0mm, board-only, no silkscreen) on every net of core,
can-card, io-card, serial-card and can-ssr, only on copper the net
already has (track, via or pour): no routing changes. Clear of foreign
copper, courtyards, all silkscreen, isolation gaps; 0.5 mm from the net's
own pads so the probe measures through the joint. Where nothing fits the
probe point is an SMD pad toe. Bottom-side test points where the parts
are on the bottom (can-ssr). DRC loop moves offenders; check_board clean
on all five boards, no reference texts moved or hidden.

tools/tptest.py: plan (net vs domain ground, across two-pin parts,
isolation between ground domains; powered.csv rail checklist) and run
(golden recording, compare with tolerance + golden spread, serial stream
from the planned probe helper or typed values, current.png step map).
docs/probe-test.md describes the workflow and the helper's interface.

Also: silk_tidy --only and board.json silk_keep; io-card place.py places
the AO row references; place.py scripts ignore TP footprints.

Co-Authored-By: Claude Opus 5.5 <noreply@anthropic.com>
Parts:
- added TP1: pour, Thl_TestPoint:TP_Probe_D1.0mm, F.Cu at (108.6, 101.6)
- added TP10: pour, Thl_TestPoint:TP_Probe_D1.0mm, F.Cu at (137.1, 126.6)
- added TP11: track, Thl_TestPoint:TP_Probe_D1.0mm, F.Cu at (158.7, 121.6)
- added TP12: track, Thl_TestPoint:TP_Probe_D1.0mm, F.Cu at (133.7, 136.6)
- added TP13: track, Thl_TestPoint:TP_Probe_D1.0mm, F.Cu at (135.2, 133.9)
- added TP14: track, Thl_TestPoint:TP_Probe_D1.0mm, F.Cu at (158.5, 138.1)
- added TP15: track, Thl_TestPoint:TP_Probe_D1.0mm, F.Cu at (168.1, 139.1)
- added TP16: track, Thl_TestPoint:TP_Probe_D1.0mm, F.Cu at (171.5, 133.4)
- added TP17: track, Thl_TestPoint:TP_Probe_D1.0mm, F.Cu at (179.0, 131.5)
- added TP18: track, Thl_TestPoint:TP_Probe_D1.0mm, F.Cu at (188.2, 136.3)
- added TP19: track, Thl_TestPoint:TP_Probe_D1.0mm, F.Cu at (102.2, 140.2)
- added TP2: track, Thl_TestPoint:TP_Probe_D1.0mm, F.Cu at (136.8, 107.1)
- added TP20: track, Thl_TestPoint:TP_Probe_D1.0mm, F.Cu at (158.7, 141.1)
- added TP21: track, Thl_TestPoint:TP_Probe_D1.0mm, F.Cu at (188.0, 149.7)
- added TP22: pour, Thl_TestPoint:TP_Probe_D1.0mm, F.Cu at (101.6, 151.6)
- added TP23: track, Thl_TestPoint:TP_Probe_D1.0mm, F.Cu at (130.8, 156.7)
- added TP24: track, Thl_TestPoint:TP_Probe_D1.0mm, F.Cu at (159.2, 159.3)
- added TP25: track, Thl_TestPoint:TP_Probe_D1.0mm, F.Cu at (172.3, 153.4)
- added TP26: track, Thl_TestPoint:TP_Probe_D1.0mm, F.Cu at (181.8, 159.1)
- added TP27: track, Thl_TestPoint:TP_Probe_D1.0mm, F.Cu at (133.0, 165.5)
- added TP28: track, Thl_TestPoint:TP_Probe_D1.0mm, F.Cu at (158.5, 169.6)
- added TP29: track, Thl_TestPoint:TP_Probe_D1.0mm, F.Cu at (168.1, 167.9)
- added TP3: track, Thl_TestPoint:TP_Probe_D1.0mm, F.Cu at (129.2, 114.5)
- added TP30: track, Thl_TestPoint:TP_Probe_D1.0mm, F.Cu at (178.9, 164.1)
- added TP31: track, Thl_TestPoint:TP_Probe_D1.0mm, F.Cu at (188.2, 168.3)
- added TP32: track, Thl_TestPoint:TP_Probe_D1.0mm, F.Cu at (122.7, 178.2)
- added TP33: track, Thl_TestPoint:TP_Probe_D1.0mm, F.Cu at (129.6, 179.2)
- added TP34: track, Thl_TestPoint:TP_Probe_D1.0mm, F.Cu at (158.0, 172.6)
- added TP35: track, Thl_TestPoint:TP_Probe_D1.0mm, F.Cu at (174.0, 178.5)
- added TP36: track, Thl_TestPoint:TP_Probe_D1.0mm, F.Cu at (185.7, 178.9)
- added TP37: track, Thl_TestPoint:TP_Probe_D1.0mm, F.Cu at (158.5, 187.6)
- added TP38: track, Thl_TestPoint:TP_Probe_D1.0mm, F.Cu at (168.1, 188.6)
- added TP39: track, Thl_TestPoint:TP_Probe_D1.0mm, F.Cu at (179.0, 181.0)
- added TP4: track, Thl_TestPoint:TP_Probe_D1.0mm, F.Cu at (134.4, 112.8)
- added TP40: track, Thl_TestPoint:TP_Probe_D1.0mm, F.Cu at (132.6, 191.9)
- added TP41: track, Thl_TestPoint:TP_Probe_D1.0mm, F.Cu at (158.7, 190.6)
- added TP5: track, Thl_TestPoint:TP_Probe_D1.0mm, F.Cu at (158.5, 118.5)
- added TP6: track, Thl_TestPoint:TP_Probe_D1.0mm, F.Cu at (168.1, 116.9)
- added TP7: track, Thl_TestPoint:TP_Probe_D1.0mm, F.Cu at (171.5, 113.9)
- added TP8: track, Thl_TestPoint:TP_Probe_D1.0mm, F.Cu at (178.9, 113.0)
- added TP9: track, Thl_TestPoint:TP_Probe_D1.0mm, F.Cu at (188.2, 119.4)

Commit message: Move core, can-card, io-card, serial-card, can-ssr, probe-helper to rev B
Rev A went to PCBWay and is tagged revA. Rev B replaces parts the Mouser
BOM check flagged (obsolete, end of life, not recommended for new designs,
or not orderable) and swaps out-of-stock passives and diodes for in-stock
equivalents. Field-only changes, same footprints, no layout change; the
reference boards (can-controller, pic-module) get the same part numbers.
The rev A order lists (DigiKey, Mouser) carry the same substitutions; the
Mouser list leaves out the T821 box headers (bought from DigiKey).

docs/rev-b-changes.md lists every change and the rev B to-dos (MAX7219 is
obsolete and must be replaced). transfer/mouser-revA.xlsx (Mouser BOM
check) consumed.

Co-Authored-By: Claude Opus 5.5 <noreply@anthropic.com>
Parts:
- FB10, FB11, FB12, FB13, FB14, FB15, FB16, FB17: value BLM31KN102SN1L -> BLM31KN102SH1L

Commit message: Rev B / rev A order: 10 uF CL31B106KAHZW6E, beads BLM31PG391SN1L
Both earlier substitutes (CL31B106KAHNNNE, BLM31KN102SH1L) are on
backorder at Mouser. CL31B106KAHZW6E has the same rating (1.4 mm tall).
The isolated-supply beads need no 1 kOhm: TI's reference uses 330 Ohm;
BLM31PG391SN1L is 390 Ohm @ 100 MHz, 2 A, 50 mOhm. Field-only changes;
order lists regenerated.

Co-Authored-By: Claude Opus 5.5 <noreply@anthropic.com>
Parts:
- FB10, FB11, FB12, FB13, FB14, FB15, FB16, FB17: value BLM31KN102SH1L -> BLM31PG391SN1L
Changed lines of the file:
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@@
 			)
 		)
-		(property "MPN" "CL31B106KAHNNNE"
+		(property "MPN" "CL31B106KAHZW6E"
 			(at 0 0 0)
 			(layer "F.Fab")
@@
 			)
 		)
-		(property "MPN" "CL31B106KAHNNNE"
+		(property "MPN" "CL31B106KAHZW6E"
 			(at 0 0 270)
 			(layer "F.Fab")
@@
 			)
 		)
-		(property "MPN" "CL31B106KAHNNNE"
+		(property "MPN" "CL31B106KAHZW6E"
 			(at 0 0 270)
 			(layer "F.Fab")
@@
 			)
 		)
-		(property "MPN" "CL31B106KAHNNNE"
+		(property "MPN" "CL31B106KAHZW6E"
 			(at 0 0 270)
 			(layer "F.Fab")
@@
 			)
 		)
-		(property "MPN" "CL31B106KAHNNNE"
+		(property "MPN" "CL31B106KAHZW6E"
 			(at 0 0 270)
 			(layer "F.Fab")
@@
 			)
 		)
-		(property "MPN" "CL31B106KAHNNNE"
+		(property "MPN" "CL31B106KAHZW6E"
 			(at 0 0 0)
 			(layer "F.Fab")
@@
 			)
 		)
-		(property "Value" "BLM31KN102SH1L"
+		(property "Value" "BLM31PG391SN1L"
 			(at 0 1.9 0)
 			(layer "F.Fab")
@@
 			)
 		)
-		(property "MPN" "BLM31KN102SH1L"
+		(property "MPN" "BLM31PG391SN1L"
 			(at 0 0 0)
 			(layer "F.Fab")
@@
 			)
 		)
-		(property "MPN" "CL31B106KAHNNNE"
+		(property "MPN" "CL31B106KAHZW6E"
 			(at 0 0 270)
 			(layer "F.Fab")
@@
 			)
 		)
-		(property "MPN" "CL31B106KAHNNNE"
+		(property "MPN" "CL31B106KAHZW6E"
 			(at 0 0 270)
 			(layer "F.Fab")
@@
 			)
 		)
-		(property "Value" "BLM31KN102SH1L"
+		(property "Value" "BLM31PG391SN1L"
 			(at 0 1.9 90)
 			(layer "F.Fab")
@@
 			)
 		)
-		(property "MPN" "BLM31KN102SH1L"
+		(property "MPN" "BLM31PG391SN1L"
 			(at 0 0 90)
 			(layer "F.Fab")
@@
 			)
 		)
-		(property "Value" "BLM31KN102SH1L"
+		(property "Value" "BLM31PG391SN1L"
 			(at 0 1.9 90)
 			(layer "F.Fab")
@@
 			)
 		)
-		(property "MPN" "BLM31KN102SH1L"
+		(property "MPN" "BLM31PG391SN1L"
 			(at 0 0 90)
 			(layer "F.Fab")
@@
 			)
 		)
-		(property "MPN" "CL31B106KAHNNNE"
+		(property "MPN" "CL31B106KAHZW6E"
 			(at 0 0 0)
 			(layer "F.Fab")
@@
 			)
 		)
-		(property "MPN" "CL31B106KAHNNNE"
+		(property "MPN" "CL31B106KAHZW6E"
 			(at 0 0 0)
 			(layer "F.Fab")
@@
 			)
 		)
-		(property "Value" "BLM31KN102SH1L"
+		(property "Value" "BLM31PG391SN1L"
 			(at 0 1.9 0)
 			(layer "F.Fab")
@@
 			)
 		)
-		(property "MPN" "BLM31KN102SH1L"
+		(property "MPN" "BLM31PG391SN1L"
 			(at 0 0 0)
 			(layer "F.Fab")
@@
 			)
 		)
-		(property "Value" "BLM31KN102SH1L"
+		(property "Value" "BLM31PG391SN1L"
 			(at 0 1.9 0)
 			(layer "F.Fab")
@@
 			)
 		)
-		(property "MPN" "BLM31KN102SH1L"
+		(property "MPN" "BLM31PG391SN1L"
 			(at 0 0 0)
 			(layer "F.Fab")
@@
 			)
 		)
-		(property "Value" "BLM31KN102SH1L"
+		(property "Value" "BLM31PG391SN1L"
 			(at 0 1.9 0)
 			(layer "F.Fab")
@@
 			)
 		)
-		(property "MPN" "BLM31KN102SH1L"
+		(property "MPN" "BLM31PG391SN1L"
 			(at 0 0 0)
 			(layer "F.Fab")
@@
 			)
 		)
-		(property "MPN" "CL31B106KAHNNNE"
+		(property "MPN" "CL31B106KAHZW6E"
 			(at 0 0 270)
 			(layer "F.Fab")
@@
 			)
 		)
-		(property "Value" "BLM31KN102SH1L"
+		(property "Value" "BLM31PG391SN1L"
 			(at 0 1.9 90)
 			(layer "F.Fab")
@@
 			)
 		)
-		(property "MPN" "BLM31KN102SH1L"
+		(property "MPN" "BLM31PG391SN1L"
 			(at 0 0 90)
 			(layer "F.Fab")
@@
 			)
 		)
-		(property "MPN" "CL31B106KAHNNNE"
+		(property "MPN" "CL31B106KAHZW6E"
 			(at 0 0 270)
 			(layer "F.Fab")
@@
 			)
 		)
-		(property "Value" "BLM31KN102SH1L"
+		(property "Value" "BLM31PG391SN1L"
 			(at 0 1.9 90)
 			(layer "F.Fab")
@@
 			)
 		)
-		(property "MPN" "BLM31KN102SH1L"
+		(property "MPN" "BLM31PG391SN1L"
 			(at 0 0 90)
 			(layer "F.Fab")

Commit message: Rev B / rev A order: ISOW1044BDFMR (ISOW1044DFMR out of stock)
Same TI part, package and pinout with basic instead of reinforced
isolation; the CAN buses are low-voltage and isolated against ground
loops, not for safety. Field-only change on can-card (and the reference
can-controller); order lists regenerated.

Co-Authored-By: Claude Opus 5.5 <noreply@anthropic.com>
Parts:
- U10, U11, U12, U13: value ISOW1044 -> ISOW1044B
Changed lines of the file:
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@@
 			)
 		)
-		(property "Value" "ISOW1044"
+		(property "Value" "ISOW1044B"
 			(at 0 7.35 0)
 			(layer "F.Fab")
@@
 			)
 		)
-		(property "MPN" "ISOW1044DFMR"
+		(property "MPN" "ISOW1044BDFMR"
 			(at 0 0 0)
 			(layer "F.Fab")
@@
 			)
 		)
-		(property "Value" "ISOW1044"
+		(property "Value" "ISOW1044B"
 			(at 0 7.35 0)
 			(layer "F.Fab")
@@
 			)
 		)
-		(property "MPN" "ISOW1044DFMR"
+		(property "MPN" "ISOW1044BDFMR"
 			(at 0 0 0)
 			(layer "F.Fab")
@@
 			)
 		)
-		(property "Value" "ISOW1044"
+		(property "Value" "ISOW1044B"
 			(at 0 7.35 0)
 			(layer "F.Fab")
@@
 			)
 		)
-		(property "MPN" "ISOW1044DFMR"
+		(property "MPN" "ISOW1044BDFMR"
 			(at 0 0 0)
 			(layer "F.Fab")
@@
 			)
 		)
-		(property "Value" "ISOW1044"
+		(property "Value" "ISOW1044B"
 			(at 0 7.35 0)
 			(layer "F.Fab")
@@
 			)
 		)
-		(property "MPN" "ISOW1044DFMR"
+		(property "MPN" "ISOW1044BDFMR"
 			(at 0 0 0)
 			(layer "F.Fab")
