File: boards/pic-module/hardware/pic-module.kicad_pcb (KiCad board)
At the start: 2 copper layers, 56 x 74 mm, 42 parts, among them J2 ICSP, J20 12V IN, J3 J3 host, J4 J4 host, J5 UART, Q1 SUD50P04-08, U1 PIC32MK1024MCM064-I/PT, U2 MCP1826S-3302E/DB, U20 TDN 5-2411WI, Y1 12MHz

Commit message: Mouser cart: SQD50P04-09L P-FET, Diotec P6SMBJ15A TVS
Out of stock: Vishay SUD50P04-08-GE3 (core Q1) -> SQD50P04-09L_GE3 and
Littelfuse SMBJ15A (12 V input TVS) -> Diotec P6SMBJ15A, same footprints,
in core, can-ssr and the can-controller/pic-module references. Logged in
docs/rev-b-changes.md; order lists regenerated. The cart as ordered is
docs/orders/mouser-cart-2026-10-12.xls.

Co-Authored-By: Claude Opus 5.5 <noreply@anthropic.com>
Parts:
- D31: value SMBJ15A -> P6SMBJ15A
- Q1: value SUD50P04-08 -> SQD50P04-09L
Changed lines of the file:
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@@
 			)
 		)
-		(property "Value" "SUD50P04-08"
+		(property "Value" "SQD50P04-09L"
 			(at 0 4.5 180)
 			(layer "F.Fab")
@@
 			)
 		)
-		(property "MPN" "SUD50P04-08-GE3"
+		(property "MPN" "SQD50P04-09L_GE3"
 			(at 0 0 180)
 			(layer "F.Fab")
@@
 			)
 		)
-		(property "Value" "SMBJ15A"
+		(property "Value" "P6SMBJ15A"
 			(at 0 3 90)
 			(layer "F.Fab")
@@
 			)
 		)
-		(property "Manufacturer" "Littelfuse"
+		(property "Manufacturer" "Diotec Semiconductor"
 			(at 0 0 90)
 			(layer "F.Fab")
@@
 			)
 		)
-		(property "MPN" "SMBJ15A"
+		(property "MPN" "P6SMBJ15A"
 			(at 0 0 90)
 			(layer "F.Fab")
